Commit message: Yeni araç STL eklendi, siyah tekerlekler kaldırıldı, URDF güncellendi

File: urdf/robot.urdf.xacro (robot description, xacro)
@@ -19,8 +19,9 @@
   <!-- ─── ŞASİ ─────────────────────────────────── -->
   <link name="base_link">
-    <visual>
+     <visual>
       <origin xyz="0 0 0" rpy="0 0 0"/>
       <geometry>
-        <box size="1.2 0.6 0.24"/>
+        <mesh filename="package://tulpar_description/meshes/tulpar_yeni.stl"
+              scale="0.001 0.001 0.001"/>
       </geometry>
       <material name="aluminium">
@@ -31,5 +32,5 @@
       <origin xyz="0 0 0" rpy="0 0 0"/>
       <geometry>
-        <box size="1.2 0.6 0.24"/>
+        <box size="1.316 1.207 0.615"/>
       </geometry>
     </collision>
@@ -49,26 +50,9 @@
     </inertial>
   </link>
-  <!-- ─── SOL ÖN TEKERLEK ──────────────────────── -->
+  <!-- Sol ön tekerlek - görünmez fizik linki -->
   <link name="wheel_fl">
-    <visual>
-      <origin xyz="0 0 0" rpy="0 0 0"/>
-      <geometry>
-        <cylinder radius="0.165" length="0.12"/>
-      </geometry>
-      <material name="dark">
-        <color rgba="0.1 0.1 0.1 1"/>
-      </material>
-    </visual>
-    <collision>
-      <geometry>
-        <cylinder radius="0.165" length="0.12"/>
-      </geometry>
-    </collision>
-    <inertial>
-      <mass value="3.5"/>
-      <inertia
-        ixx="0.024"  ixy="0"  ixz="0"
-        iyy="0.024"  iyz="0"
-        izz="0.048"/>
+    <inertial>
+      <mass value="3.5"/>
+      <inertia ixx="0.024" ixy="0" ixz="0" iyy="0.024" iyz="0" izz="0.048"/>
     </inertial>
   </link>
@@ -76,31 +60,13 @@
     <parent link="base_link"/>
     <child link="wheel_fl"/>
-    <!-- x: dingil/2=0.4, y: iz/2=0.52, z: tekerlek tabanı -->
     <origin xyz="0.4 0.58 -0.24" rpy="-1.5708 0 0"/>
     <axis xyz="0 0 1"/>
     <dynamics damping="0.1" friction="0.5"/>
   </joint>
-  <!-- ─── SOL ARKA TEKERLEK ─────────────────────── -->
+  <!-- Sol arka tekerlek -->
   <link name="wheel_rl">
-    <visual>
-      <origin xyz="0 0 0" rpy="0 0 0"/>
-      <geometry>
-        <cylinder radius="0.165" length="0.12"/>
-      </geometry>
-      <material name="dark">
-        <color rgba="0.1 0.1 0.1 1"/>
-      </material>
-    </visual>
-    <collision>
-      <geometry>
-        <cylinder radius="0.165" length="0.12"/>
-      </geometry>
-    </collision>
-    <inertial>
-      <mass value="3.5"/>
-      <inertia
-        ixx="0.024"  ixy="0"  ixz="0"
-        iyy="0.024"  iyz="0"
-        izz="0.048"/>
+    <inertial>
+      <mass value="3.5"/>
+      <inertia ixx="0.024" ixy="0" ixz="0" iyy="0.024" iyz="0" izz="0.048"/>
     </inertial>
   </link>
@@ -112,26 +78,9 @@
     <dynamics damping="0.1" friction="0.5"/>
   </joint>
-  <!-- ─── SAĞ ÖN TEKERLEK ──────────────────────── -->
+  <!-- Sağ ön tekerlek -->
   <link name="wheel_fr">
-    <visual>
-      <origin xyz="0 0 0" rpy="0 0 0"/>
-      <geometry>
-        <cylinder radius="0.165" length="0.12"/>
-      </geometry>
-      <material name="dark">
-        <color rgba="0.1 0.1 0.1 1"/>
-      </material>
-    </visual>
-    <collision>
-      <geometry>
-        <cylinder radius="0.165" length="0.12"/>
-      </geometry>
-    </collision>
-    <inertial>
-      <mass value="3.5"/>
-      <inertia
-        ixx="0.024"  ixy="0"  ixz="0"
-        iyy="0.024"  iyz="0"
-        izz="0.048"/>
+    <inertial>
+      <mass value="3.5"/>
+      <inertia ixx="0.024" ixy="0" ixz="0" iyy="0.024" iyz="0" izz="0.048"/>
     </inertial>
   </link>
@@ -143,26 +92,9 @@
     <dynamics damping="0.1" friction="0.5"/>
   </joint>
-  <!-- ─── SAĞ ARKA TEKERLEK ─────────────────────── -->
+  <!-- Sağ arka tekerlek -->
   <link name="wheel_rr">
-    <visual>
-      <origin xyz="0 0 0" rpy="0 0 0"/>
-      <geometry>
-        <cylinder radius="0.165" length="0.12"/>
-      </geometry>
-      <material name="dark">
-        <color rgba="0.1 0.1 0.1 1"/>
-      </material>
-    </visual>
-    <collision>
-      <geometry>
-        <cylinder radius="0.165" length="0.12"/>
-      </geometry>
-    </collision>
-    <inertial>
-      <mass value="3.5"/>
-      <inertia
-        ixx="0.024"  ixy="0"  ixz="0"
-        iyy="0.024"  iyz="0"
-        izz="0.048"/>
+    <inertial>
+      <mass value="3.5"/>
+      <inertia ixx="0.024" ixy="0" ixz="0" iyy="0.024" iyz="0" izz="0.048"/>
     </inertial>
   </link>
