Commit message: URDF strateji pivotu: Zehra'nin feature/zehra-faz1-gun1 URDF+mesh yaklasimi temel alindi
Mekanik ekip orijinal tulpar_ika_assembly.stl'in Blender'da eksiksiz
oldugunu dogruladi - detay kaybi bizim decimation pipeline'imizdaydi
(govde/teker v2/v3 mesh'leri ve ilgili yaklasim terk edildi, silindi).

Zehra'nin urdf/robot.urdf.xacro + ham tulpar_ika_assembly.stl (149MB,
Git LFS ile - GitHub'in 100MB limitini asiyor) kendi dosyalarimizin
yerine kondu; sadece fiziksel parametreler (1200x450x245mm, 64kg,
780mm dingil, 1060mm iz, 200mm tekerlek yaricapi, yeniden hesaplanan
analitik kutu inertia) mekanik ekipten guncellendi. Sensor link
isimleri Zehra'nin adlandirmasiyla birlesti (d435i_link, rear_camera_link
- gercek Gazebo sensor plugin'lerine bagli).

.gitattributes eklendi: *.stl artik Git LFS uzerinden takip ediliyor
(Zehra'nin branch'iyle tutarli). Sadece bundan sonraki .stl'ler icin
gecerli, tulpar_yeni.stl gibi mevcut tracked dosyalar etkilenmedi.

CLAUDE.md guncellendi: yeni durum, bilinen sorunlar (gazebo.launch.py
bridge topic uyumsuzlugu) ve Gun 4 ilerleme notu eklendi.

File: urdf/robot.urdf.xacro (robot description, xacro)
@@ -1,59 +1,59 @@
 <?xml version="1.0"?>
 <robot name="tulpar_robot" xmlns:xacro="http://www.ros.org/wiki/xacro">
-  <!-- ═══════════════════════════════════════════════
-       TULPAR İKA — URDF v2.1 (geometri duzeltildi)
-       Şasi     : 1200 x 600 x 240 mm, 62 kg
-       Tekerlek : Ø330 mm (r=0.165 m)
-       İz gen.  : 1040 mm
-       Dingil   : 800 mm
-       ═══════════════════════════════════════════════ -->
+  <material name="aluminium">
+    <color rgba="0.75 0.75 0.75 1.0"/>
+  </material>
+  <material name="black">
+    <color rgba="0.1 0.1 0.1 1.0"/>
+  </material>
+  <material name="camera_blue">
+    <color rgba="0.0 0.2 0.8 1.0"/>
+  </material>
+  <material name="sensor_gray">
+    <color rgba="0.3 0.3 0.3 1.0"/>
+  </material>
   <link name="base_footprint"/>
-  <!-- base_link tekerlek ekseni hizasinda (z=0.165) -->
   <joint name="base_joint" type="fixed">
     <parent link="base_footprint"/>
     <child link="base_link"/>
-    <origin xyz="0 0 0.165" rpy="0 0 0"/>
-  </joint>
-  <!-- ─── ŞASİ ─────────────────────────────────── -->
+    <!-- z=0.200: yeni tekerlek yaricapi ile tutarli (base_link tekerlek
+         ekseni hizasinda olmali) -->
+    <origin xyz="0 0 0.200" rpy="0 0 0"/>
+  </joint>
   <link name="base_link">
     <visual>
       <origin xyz="0.600 -0.300 0.110" rpy="0 0 1.5708"/>
       <geometry>
-        <mesh filename="package://tulpar_description/meshes/tulpar_yeni.stl"
-              scale="0.001 0.001 0.001"/>
-      </geometry>
-      <material name="aluminium">
-        <color rgba="0.75 0.75 0.75 1"/>
-      </material>
+        <mesh filename="package://tulpar_description/meshes/tulpar_ika_assembly.stl" scale="0.001 0.001 0.001"/>
+      </geometry>
+      <material name="aluminium"/>
     </visual>
     <collision>
-      <origin xyz="0 0 0.1925" rpy="0 0 0"/>
-      <geometry>
-        <box size="1.316 1.207 0.615"/>
+      <!-- z=0.187: gercek (transform uygulanmis) mesh bbox merkezinden turetilen
+           deger, ADIM2/URDF v3.0 calismasindan korunuyor -->
+      <origin xyz="0 0 0.187" rpy="0 0 0"/>
+      <geometry>
+        <box size="1.200 0.450 0.245"/>
       </geometry>
     </collision>
     <inertial>
-      <mass value="60.0"/>
+      <mass value="64.0"/>
       <origin xyz="0 0 0" rpy="0 0 0"/>
-      <inertia
-        ixx="8.520"   ixy="0.0"  ixz="0.0"
-        iyy="22.140"  iyz="0.0"
-        izz="27.180"/>
-    </inertial>
-  </link>
-  <!-- ─── TEKERLEKLER (collision eklendi) ──────── -->
-  <xacro:macro name="tekerlek" params="isim x y">
-    <link name="${isim}">
+      <!-- Analitik kutu (1.2x0.45x0.245m, 64.0kg) - fiziksel olarak garantili
+           gecerli (ucgen esitsizligi tam saglaniyor) -->
+      <inertia ixx="1.4001" ixy="0.0" ixz="0.0" iyy="8.0001" iyz="0.0" izz="8.7600"/>
+    </inertial>
+  </link>
+  <xacro:macro name="wheel" params="name x y">
+    <link name="${name}">
       <visual>
-        <origin xyz="0 0 0" rpy="0 0 0"/>
         <geometry>
-          <cylinder radius="0.165" length="0.12"/>
+          <cylinder radius="0.200" length="0.12"/>
         </geometry>
-        <material name="black"><color rgba="0.1 0.1 0.1 1"/></material>
+        <material name="black"/>
       </visual>
       <collision>
-        <origin xyz="0 0 0" rpy="0 0 0"/>
         <geometry>
-          <cylinder radius="0.165" length="0.12"/>
+          <cylinder radius="0.200" length="0.12"/>
         </geometry>
       </collision>
@@ -63,8 +63,7 @@
       </inertial>
     </link>
-    <joint name="joint_${isim}" type="continuous">
+    <joint name="joint_${name}" type="continuous">
       <parent link="base_link"/>
-      <child link="${isim}"/>
-      <!-- z=0: tekerlek merkezi base_link ile ayni hizada (zeminden 0.165m) -->
+      <child link="${name}"/>
       <origin xyz="${x} ${y} 0" rpy="-1.5708 0 0"/>
       <axis xyz="0 0 1"/>
@@ -72,17 +71,18 @@
     </joint>
   </xacro:macro>
-  <xacro:tekerlek isim="wheel_fl" x="0.4"  y="0.52"/>
-  <xacro:tekerlek isim="wheel_rl" x="-0.4" y="0.52"/>
-  <xacro:tekerlek isim="wheel_fr" x="0.4"  y="-0.52"/>
-  <xacro:tekerlek isim="wheel_rr" x="-0.4" y="-0.52"/>
-  <!-- ─── LİDAR ─────────────────────────────────── -->
+  <xacro:wheel name="wheel_fl" x="0.39" y="0.53"/>
+  <xacro:wheel name="wheel_rl" x="-0.39" y="0.53"/>
+  <xacro:wheel name="wheel_fr" x="0.39" y="-0.53"/>
+  <xacro:wheel name="wheel_rr" x="-0.39" y="-0.53"/>
   <link name="lidar_link">
     <visual>
-      <geometry><cylinder radius="0.04" length="0.04"/></geometry>
-      <material name="lidar_black"><color rgba="0 0 0 1"/></material>
-    </visual>
-    <inertial>
-      <mass value="0.18"/>
-      <inertia ixx="0.001" ixy="0" ixz="0" iyy="0.001" iyz="0" izz="0.001"/>
+      <geometry>
+        <cylinder radius="0.05" length="0.06"/>
+      </geometry>
+      <material name="sensor_gray"/>
+    </visual>
+    <inertial>
+      <mass value="0.25"/>
+      <inertia ixx="0.0015" ixy="0" ixz="0" iyy="0.0015" iyz="0" izz="0.0015"/>
     </inertial>
   </link>
@@ -90,60 +90,131 @@
     <parent link="base_link"/>
     <child link="lidar_link"/>
-    <origin xyz="0.3 0 0.4" rpy="0 0 0"/>
-  </joint>
-  <!-- ─── REALSENSE D455 ────────────────────────── -->
-  <link name="camera_link">
-    <visual>
-      <geometry><box size="0.09 0.025 0.025"/></geometry>
-      <material name="cam_blue"><color rgba="0.0 0.2 0.8 1"/></material>
+    <origin xyz="0.30 0.0 0.40" rpy="0 0 0"/>
+  </joint>
+  <link name="laser_frame"/>
+  <joint name="laser_frame_joint" type="fixed">
+    <parent link="lidar_link"/>
+    <child link="laser_frame"/>
+    <origin xyz="0 0 0" rpy="0 0 0"/>
+  </joint>
+  <link name="d435i_link">
+    <visual>
+      <geometry>
+        <box size="0.09 0.025 0.025"/>
+      </geometry>
+      <material name="camera_blue"/>
+    </visual>
+    <inertial>
+      <mass value="0.08"/>
+      <inertia ixx="0.001" ixy="0" ixz="0" iyy="0.001" iyz="0" izz="0.001"/>
+    </inertial>
+  </link>
+  <joint name="d435i_joint" type="fixed">
+    <parent link="base_link"/>
+    <child link="d435i_link"/>
+    <origin xyz="0.62 0.0 0.20" rpy="0 0 0"/>
+  </joint>
+  <link name="d435i_color_frame"/>
+  <joint name="d435i_color_joint" type="fixed">
+    <parent link="d435i_link"/>
+    <child link="d435i_color_frame"/>
+    <origin xyz="0 0 0" rpy="0 0 0"/>
+  </joint>
+  <link name="d435i_color_optical_frame"/>
+  <joint name="d435i_color_optical_joint" type="fixed">
+    <parent link="d435i_color_frame"/>
+    <child link="d435i_color_optical_frame"/>
+    <origin xyz="0 0 0" rpy="-1.5708 0 -1.5708"/>
+  </joint>
+  <link name="d435i_depth_frame"/>
+  <joint name="d435i_depth_joint" type="fixed">
+    <parent link="d435i_link"/>
+    <child link="d435i_depth_frame"/>
+    <origin xyz="0 0 0" rpy="0 0 0"/>
+  </joint>
+  <link name="d435i_depth_optical_frame"/>
+  <joint name="d435i_depth_optical_joint" type="fixed">
+    <parent link="d435i_depth_frame"/>
+    <child link="d435i_depth_optical_frame"/>
+    <origin xyz="0 0 0" rpy="-1.5708 0 -1.5708"/>
+  </joint>
+  <link name="rpi_hq_camera_link">
+    <visual>
+      <geometry>
+        <box size="0.038 0.038 0.018"/>
+      </geometry>
+      <material name="sensor_gray"/>
+    </visual>
+    <inertial>
+      <mass value="0.05"/>
+      <inertia ixx="0.0004" ixy="0" ixz="0" iyy="0.0004" iyz="0" izz="0.0004"/>
+    </inertial>
+  </link>
+  <joint name="rpi_hq_camera_joint" type="fixed">
+    <parent link="base_link"/>
+    <child link="rpi_hq_camera_link"/>
+    <origin xyz="0.58 0.0 0.28" rpy="0 0 0"/>
+  </joint>
+  <link name="rpi_hq_camera_optical_frame"/>
+  <joint name="rpi_hq_camera_optical_joint" type="fixed">
+    <parent link="rpi_hq_camera_link"/>
+    <child link="rpi_hq_camera_optical_frame"/>
+    <origin xyz="0 0 0" rpy="-1.5708 0 -1.5708"/>
+  </joint>
+  <link name="rear_camera_link">
+    <visual>
+      <geometry>
+        <box size="0.06 0.03 0.03"/>
+      </geometry>
+      <material name="sensor_gray"/>
     </visual>
     <inertial>
       <mass value="0.07"/>
-      <inertia ixx="0.001" ixy="0" ixz="0" iyy="0.001" iyz="0" izz="0.001"/>
-    </inertial>
-  </link>
-  <joint name="camera_joint" type="fixed">
+      <inertia ixx="0.0008" ixy="0" ixz="0" iyy="0.0008" iyz="0" izz="0.0008"/>
+    </inertial>
+  </link>
+  <joint name="rear_camera_joint" type="fixed">
     <parent link="base_link"/>
-    <child link="camera_link"/>
-    <origin xyz="0.62 0 0.2" rpy="0 0 0"/>
-  </joint>
-  <!-- ═══════════════════════════════════════════════
-       GAZEBO PLUGIN'LERİ
-       ═══════════════════════════════════════════════ -->
+    <child link="rear_camera_link"/>
+    <origin xyz="-0.58 0.0 0.28" rpy="0 0 3.14159"/>
+  </joint>
+  <link name="rear_camera_optical_frame"/>
+  <joint name="rear_camera_optical_joint" type="fixed">
+    <parent link="rear_camera_link"/>
+    <child link="rear_camera_optical_frame"/>
+    <origin xyz="0 0 0" rpy="-1.5708 0 -1.5708"/>
+  </joint>
   <gazebo>
-    <plugin filename="gz-sim-joint-state-publisher-system"
-            name="gz::sim::systems::JointStatePublisher">
+    <plugin filename="gz-sim-joint-state-publisher-system" name="gz::sim::systems::JointStatePublisher">
       <topic>/joint_states</topic>
     </plugin>
   </gazebo>
   <gazebo>
-    <plugin filename="gz-sim-diff-drive-system"
-            name="gz::sim::systems::DiffDrive">
+    <plugin filename="gz-sim-diff-drive-system" name="gz::sim::systems::DiffDrive">
       <left_joint>joint_wheel_fl</left_joint>
       <left_joint>joint_wheel_rl</left_joint>
       <right_joint>joint_wheel_fr</right_joint>
       <right_joint>joint_wheel_rr</right_joint>
-      <wheel_separation>1.04</wheel_separation>
-      <wheel_radius>0.165</wheel_radius>
-      <max_linear_velocity>0.785</max_linear_velocity>
-      <max_angular_velocity>7.854</max_angular_velocity>
-      <max_wheel_torque>21.6</max_wheel_torque>
-      <max_linear_acceleration>5.0</max_linear_acceleration>
+      <wheel_separation>1.06</wheel_separation>
+      <wheel_radius>0.200</wheel_radius>
+      <max_linear_velocity>1.0</max_linear_velocity>
+      <max_angular_velocity>3.0</max_angular_velocity>
+      <max_wheel_torque>25.0</max_wheel_torque>
+      <max_linear_acceleration>2.0</max_linear_acceleration>
       <topic>/cmd_vel</topic>
       <odom_topic>/odom</odom_topic>
       <frame_id>odom</frame_id>
       <child_frame_id>base_footprint</child_frame_id>
-      <odom_publish_frequency>50</odom_publish_frequency>
+      <odom_publish_frequency>30</odom_publish_frequency>
     </plugin>
   </gazebo>
   <gazebo reference="lidar_link">
-    <sensor name="rplidar_s2" type="gpu_lidar">
-      <update_rate>10</update_rate>
-      <topic>scan</topic>
-      <gz_frame_id>lidar_link</gz_frame_id>
+    <sensor name="ydlidar_tg30" type="gpu_lidar">
+      <update_rate>5</update_rate>
+      <topic>/scan</topic>
       <lidar>
         <scan>
           <horizontal>
-            <samples>800</samples>
+            <samples>720</samples>
             <resolution>1</resolution>
             <min_angle>-3.14159</min_angle>
@@ -154,43 +225,94 @@
           <min>0.05</min>
           <max>30.0</max>
-          <resolution>0.03</resolution>
+          <resolution>0.01</resolution>
         </range>
       </lidar>
+      <always_on>true</always_on>
+      <visualize>false</visualize>
     </sensor>
   </gazebo>
-  <gazebo reference="camera_link">
-    <sensor name="realsense_d455" type="depth_camera">
-      <update_rate>30</update_rate>
-      <topic>camera/depth</topic>
-      <gz_frame_id>camera_link</gz_frame_id>
+  <gazebo reference="d435i_link">
+    <sensor name="d435i_depth" type="depth_camera">
+      <update_rate>10</update_rate>
+      <topic>/d435i/depth/image_raw</topic>
       <camera>
-        <horizontal_fov>1.5708</horizontal_fov>
+        <horizontal_fov>1.5184</horizontal_fov>
         <image>
-          <width>848</width>
+          <width>640</width>
           <height>480</height>
           <format>R8G8B8</format>
         </image>
         <clip>
-          <near>0.4</near>
-          <far>6.0</far>
+          <near>0.20</near>
+          <far>10.0</far>
         </clip>
       </camera>
+      <always_on>true</always_on>
+      <visualize>false</visualize>
     </sensor>
   </gazebo>
+  <gazebo reference="rpi_hq_camera_link">
+    <sensor name="rpi_hq_camera" type="camera">
+      <update_rate>10</update_rate>
+      <topic>/rpi_hq_camera/image_raw</topic>
+      <camera>
+        <horizontal_fov>0.6606</horizontal_fov>
+        <image>
+          <width>640</width>
+          <height>480</height>
+          <format>R8G8B8</format>
+        </image>
+        <clip>
+          <near>0.10</near>
+          <far>100.0</far>
+        </clip>
+      </camera>
+      <always_on>true</always_on>
+      <visualize>false</visualize>
+    </sensor>
+  </gazebo>
+  <gazebo reference="rear_camera_link">
+    <sensor name="rear_camera" type="camera">
+      <update_rate>5</update_rate>
+      <topic>/rear_camera/image_raw</topic>
+      <camera>
+        <horizontal_fov>1.5708</horizontal_fov>
+        <image>
+          <width>640</width>
+          <height>480</height>
+          <format>R8G8B8</format>
+        </image>
+        <clip>
+          <near>0.10</near>
+          <far>100.0</far>
+        </clip>
+      </camera>
+      <always_on>true</always_on>
+      <visualize>false</visualize>
+    </sensor>
+  </gazebo>
   <gazebo reference="wheel_fl">
-    <mu1>1.0</mu1><mu2>1.0</mu2>
-    <kp>1000000.0</kp><kd>1.0</kd>
+    <mu1>1.0</mu1>
+    <mu2>1.0</mu2>
+    <kp>1000000.0</kp>
+    <kd>1.0</kd>
   </gazebo>
   <gazebo reference="wheel_rl">
-    <mu1>1.0</mu1><mu2>1.0</mu2>
-    <kp>1000000.0</kp><kd>1.0</kd>
+    <mu1>1.0</mu1>
+    <mu2>1.0</mu2>
+    <kp>1000000.0</kp>
+    <kd>1.0</kd>
   </gazebo>
   <gazebo reference="wheel_fr">
-    <mu1>1.0</mu1><mu2>1.0</mu2>
-    <kp>1000000.0</kp><kd>1.0</kd>
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
Commit message: Cifte tekerlek gorsel cakismasi duzeltildi + D435if bridge topic guncellendi
GOREV 1 - Tekerlek geometrisi:
tulpar_ika_assembly.stl'den SADECE gomulu eski tekerlek geometrisi
(4 kosede 16 parca, [616,4238,4434,7844] face imzasiyla kesin
eslestirildi) cikarildi, govdeye/decimation'a dokunulmadi. Sonuc
meshes/tulpar_ika_assembly_tekersiz.stl (149MB -> 139MB). Orijinal
dosya korundu, URDF yeni dosyaya yonlendirildi.

Ilk denemede gevsek filtre (sadece ">=2 katman" kurali) 8 fazladan
yapisal parcayi (sasi raylari, suspansiyon braketleri, bir sensor
plakasi) da yanlislikla tekerlek sanip cikarmisti - tespit edilip
siki imza-eslestirmeyle (tam 4 kose, ayni face-sayisi deseni)
duzeltildi.

GOREV 2 - Bridge topic guncellemesi:
Zehra'nin dogruladigi gercek calisan D435if topic isimlerine gecildi:
/d435if/depth/image_raw, /d435if/depth/camera_info,
/d435if/depth/image_raw/points. Onceden URDF'nin kendi sensor topic'i
(/d435i/...) ile bridge'in bekledigi isim (/camera/...) birbirinden
tamamen kopuktu - ikisi de düzeltildi (urdf/robot.urdf.xacro +
launch/gazebo.launch.py). rtabmap.launch.py yorumlari guncellendi.

Gazebo testiyle dogrulandi: tekerlekler cakismadan oturuyor, 3 kamera
topic'i de gercek veri akitiyor (ros2 topic echo --once ile teyit
edildi). CLAUDE.md'ye kamera routing karar tablosu eklendi.

File: urdf/robot.urdf.xacro (robot description, xacro)
@@ -25,5 +25,5 @@
       <origin xyz="0.600 -0.300 0.110" rpy="0 0 1.5708"/>
       <geometry>
-        <mesh filename="package://tulpar_description/meshes/tulpar_ika_assembly.stl" scale="0.001 0.001 0.001"/>
+        <mesh filename="package://tulpar_description/meshes/tulpar_ika_assembly_tekersiz.stl" scale="0.001 0.001 0.001"/>
       </geometry>
       <material name="aluminium"/>
@@ -235,5 +235,7 @@
     <sensor name="d435i_depth" type="depth_camera">
       <update_rate>10</update_rate>
-      <topic>/d435i/depth/image_raw</topic>
+      <!-- Zehra'nin dogruladigi calisan topic adi: d435if (link adi d435i_link
+           kaliyor, sadece topic ismi hedef donanim adiyla (D435if) eslesiyor) -->
+      <topic>/d435if/depth/image_raw</topic>
       <camera>
         <horizontal_fov>1.5184</horizontal_fov>

Commit message: d435i_link -> d435if_link rename: URDF link/joint isimleri donanim ve bridge topic adiyla hizalandi
Zehra'nin feature/zehra-slalom-core branch'inde onerilen rename onaylandi
(D435if donanim adiyla ve zaten var olan /d435if/depth/... bridge topic
isimleriyle tutarli). urdf/robot.urdf.xacro'daki tum ilgili link/joint/
gazebo-reference isimleri tasindi, artik gereksiz aciklama yorumu
silindi, launch/rtabmap.launch.py'deki yorum guncellendi. xacro ile
derlenip TF agacinin bozulmadigi dogrulandi. CLAUDE.md guncel-durum
satirlari ve BILEREK MERGE EDILMEYENLER listesi guncellendi.

File: urdf/robot.urdf.xacro (robot description, xacro)
@@ -98,5 +98,5 @@
     <origin xyz="0 0 0" rpy="0 0 0"/>
   </joint>
-  <link name="d435i_link">
+  <link name="d435if_link">
     <visual>
       <geometry>
@@ -110,31 +110,31 @@
     </inertial>
   </link>
-  <joint name="d435i_joint" type="fixed">
+  <joint name="d435if_joint" type="fixed">
     <parent link="base_link"/>
-    <child link="d435i_link"/>
+    <child link="d435if_link"/>
     <origin xyz="0.62 0.0 0.20" rpy="0 0 0"/>
   </joint>
-  <link name="d435i_color_frame"/>
-  <joint name="d435i_color_joint" type="fixed">
-    <parent link="d435i_link"/>
-    <child link="d435i_color_frame"/>
+  <link name="d435if_color_frame"/>
+  <joint name="d435if_color_joint" type="fixed">
+    <parent link="d435if_link"/>
+    <child link="d435if_color_frame"/>
     <origin xyz="0 0 0" rpy="0 0 0"/>
   </joint>
-  <link name="d435i_color_optical_frame"/>
-  <joint name="d435i_color_optical_joint" type="fixed">
-    <parent link="d435i_color_frame"/>
-    <child link="d435i_color_optical_frame"/>
+  <link name="d435if_color_optical_frame"/>
+  <joint name="d435if_color_optical_joint" type="fixed">
+    <parent link="d435if_color_frame"/>
+    <child link="d435if_color_optical_frame"/>
     <origin xyz="0 0 0" rpy="-1.5708 0 -1.5708"/>
   </joint>
-  <link name="d435i_depth_frame"/>
-  <joint name="d435i_depth_joint" type="fixed">
-    <parent link="d435i_link"/>
-    <child link="d435i_depth_frame"/>
+  <link name="d435if_depth_frame"/>
+  <joint name="d435if_depth_joint" type="fixed">
+    <parent link="d435if_link"/>
+    <child link="d435if_depth_frame"/>
     <origin xyz="0 0 0" rpy="0 0 0"/>
   </joint>
-  <link name="d435i_depth_optical_frame"/>
-  <joint name="d435i_depth_optical_joint" type="fixed">
-    <parent link="d435i_depth_frame"/>
-    <child link="d435i_depth_optical_frame"/>
+  <link name="d435if_depth_optical_frame"/>
+  <joint name="d435if_depth_optical_joint" type="fixed">
+    <parent link="d435if_depth_frame"/>
+    <child link="d435if_depth_optical_frame"/>
     <origin xyz="0 0 0" rpy="-1.5708 0 -1.5708"/>
   </joint>
@@ -232,9 +232,7 @@
     </sensor>
   </gazebo>
-  <gazebo reference="d435i_link">
-    <sensor name="d435i_depth" type="depth_camera">
+  <gazebo reference="d435if_link">
+    <sensor name="d435if_depth" type="depth_camera">
       <update_rate>10</update_rate>
-      <!-- Zehra'nin dogruladigi calisan topic adi: d435if (link adi d435i_link
-           kaliyor, sadece topic ismi hedef donanim adiyla (D435if) eslesiyor) -->
       <topic>/d435if/depth/image_raw</topic>
       <camera>

Commit message: Sensor montaj konumlari Zehra'nin feature/zehra-slalom-core degerleriyle guncellendi
lidar/d435if/rpi_hq_camera origin xyz degerleri (274f4f1) alindi -
uc sensor de one/yukari toplanmis, muhtemelen guncel sensor
direk/braket tasarimini yansitiyor. xacro ile derlenip dogrulandi,
Gazebo'da FOV/gorsel testi henuz yapilmadi.

File: urdf/robot.urdf.xacro (robot description, xacro)
@@ -90,5 +90,5 @@
     <parent link="base_link"/>
     <child link="lidar_link"/>
-    <origin xyz="0.30 0.0 0.40" rpy="0 0 0"/>
+    <origin xyz="0.58 -0.015 0.61" rpy="0 0 0"/>
   </joint>
   <link name="laser_frame"/>
@@ -113,5 +113,5 @@
     <parent link="base_link"/>
     <child link="d435if_link"/>
-    <origin xyz="0.62 0.0 0.20" rpy="0 0 0"/>
+    <origin xyz="0.58 0.0 0.53" rpy="0 0 0"/>
   </joint>
   <link name="d435if_color_frame"/>
@@ -154,5 +154,5 @@
     <parent link="base_link"/>
     <child link="rpi_hq_camera_link"/>
-    <origin xyz="0.58 0.0 0.28" rpy="0 0 0"/>
+    <origin xyz="0.58 -0.03 0.58" rpy="0 0 0"/>
   </joint>
   <link name="rpi_hq_camera_optical_frame"/>
