Commit message: Tekerlek yaricapi govdeyle orantisiz bulundu, kendi olcumumuzle duzeltildi
wheel_radius=0.200 (primitive silindir + DiffDrive plugin) hicbir zaman
mekanik ekiple netlesmis bir deger degildi (Key Physical Parameters
notunda "Zehra'nin orijinal degerleri, henuz netlesmedi" diye isaretliydi).
Kullanici Gazebo'da tekerleklerin govdeye gore cok buyuk durdugunu fark
etti, ekran goruntusuyle dogrulandi.

Kok neden: mekanik ekibin dogruladigi gercek CAD montajindan (Gun 4,
"cifte tekerlek" duzeltmesi sirasinda) gomulu eski tekerlek geometrisi
olculmustu - ~166mm yaricap. Bu elimizdeki tek gercekten CAD-dogrulanmis
tekerlek olcusu. wheel_radius 0.200->0.166 (silindir visual+collision,
DiffDrive plugin, base_joint z-offset). Gazebo'da tekrar test edildi,
oranti duzeldi.

File: urdf/robot.urdf.xacro (robot description, xacro)
@@ -17,7 +17,9 @@
     <parent link="base_footprint"/>
     <child link="base_link"/>
-    <!-- z=0.200: yeni tekerlek yaricapi ile tutarli (base_link tekerlek
-         ekseni hizasinda olmali) -->
-    <origin xyz="0 0 0.200" rpy="0 0 0"/>
+    <!-- z=0.166: gercek tekerlek yaricapi (govde mesh'inden - tulpar_ika_assembly.stl
+         icindeki gomulu eski tekerlek geometrisinin olcumu, bkz. "cifte tekerlek"
+         notu - 0.200 degeri Zehra'nin dogrulanmamis DiffDrive degeriydi, govde
+         ile orantisiz gorunuyordu, 17 Temmuz'da duzeltildi) -->
+    <origin xyz="0 0 0.166" rpy="0 0 0"/>
   </joint>
   <link name="base_link">
@@ -49,5 +51,5 @@
       <visual>
         <geometry>
-          <cylinder radius="0.200" length="0.12"/>
+          <cylinder radius="0.166" length="0.12"/>
         </geometry>
         <material name="black"/>
@@ -55,5 +57,5 @@
       <collision>
         <geometry>
-          <cylinder radius="0.200" length="0.12"/>
+          <cylinder radius="0.166" length="0.12"/>
         </geometry>
       </collision>
@@ -197,5 +199,5 @@
       <right_joint>joint_wheel_rr</right_joint>
       <wheel_separation>1.06</wheel_separation>
-      <wheel_radius>0.200</wheel_radius>
+      <wheel_radius>0.166</wheel_radius>
       <max_linear_velocity>1.0</max_linear_velocity>
       <max_angular_velocity>3.0</max_angular_velocity>
