Commit message: Araç görsel düzeltmesi: STL mirror, yön ve rampa girişi
- STL tulpar_yeni.stl X ekseninde aynalandı (taret önden sağda)
- URDF ve tüm SDF dünyalarında mesh rotasyonu +90°, offset 0.600 -0.300 olarak güncellendi
- s01_robotlu_world.sdf: rampa tabanı 5cm yere gömüldü (z:0.203→0.153) — ODE adım sorunu giderildi
- s02_hedef_world.sdf: yeni S-02 test dünyası eklendi
- e02_duz_world.sdf: yeni E-02 test dünyası eklendi
- test_kanit/S01 ve S02: tam parkur ve hedef tespit test scriptleri eklendi
- E-02 test kanıt dosyaları güncellendi

Co-Authored-By: Claude Sonnet 4.6 <noreply@anthropic.com>

File: urdf/robot.urdf.xacro (robot description, xacro)
@@ -2,23 +2,21 @@
 <robot name="tulpar_robot" xmlns:xacro="http://www.ros.org/wiki/xacro">
   <!-- ═══════════════════════════════════════════════
-       TULPAR İKA — URDF v2.0
+       TULPAR İKA — URDF v2.1 (geometri duzeltildi)
        Şasi     : 1200 x 600 x 240 mm, 62 kg
        Tekerlek : Ø330 mm (r=0.165 m)
        İz gen.  : 1040 mm
        Dingil   : 800 mm
-       Max hız  : 0.785 m/s | Max tork: 21.6 Nm
        ═══════════════════════════════════════════════ -->
-  <!-- Zemin referans noktası -->
   <link name="base_footprint"/>
+  <!-- base_link tekerlek ekseni hizasinda (z=0.165) -->
   <joint name="base_joint" type="fixed">
     <parent link="base_footprint"/>
     <child link="base_link"/>
-    <!-- Ağırlık merkezi yüksekliği ~240mm -->
-    <origin xyz="0 0 0.24" rpy="0 0 0"/>
+    <origin xyz="0 0 0.165" rpy="0 0 0"/>
   </joint>
   <!-- ─── ŞASİ ─────────────────────────────────── -->
   <link name="base_link">
-     <visual>
-      <origin xyz="0 0 0" rpy="0 0 0"/>
+    <visual>
+      <origin xyz="0.600 -0.300 0.110" rpy="0 0 1.5708"/>
       <geometry>
         <mesh filename="package://tulpar_description/meshes/tulpar_yeni.stl"
@@ -30,5 +28,5 @@
     </visual>
     <collision>
-      <origin xyz="0 0 0" rpy="0 0 0"/>
+      <origin xyz="0 0 0.1425" rpy="0 0 0"/>
       <geometry>
         <box size="1.316 1.207 0.615"/>
@@ -36,79 +34,51 @@
     </collision>
     <inertial>
-      <!-- 62 kg, dikdörtgen kutu inertia -->
-     <mass value="60.0"/>
+      <mass value="60.0"/>
       <origin xyz="0 0 0" rpy="0 0 0"/>
       <inertia
-        ixx="2.100"  ixy="0.0"  ixz="0.0"
-        iyy="7.920"  iyz="0.0"
-        izz="9.300"/>
-      <!--
-        ixx = 60/12*(0.24²+0.6²)  = 2.100
-        iyy = 60/12*(1.2²+0.6²)   = 7.920
-        izz = 60/12*(1.2²+0.24²)  = 9.300
-      -->
+        ixx="8.520"   ixy="0.0"  ixz="0.0"
+        iyy="22.140"  iyz="0.0"
+        izz="27.180"/>
     </inertial>
   </link>
-  <!-- Sol ön tekerlek - görünmez fizik linki -->
-  <link name="wheel_fl">
-    <inertial>
-      <mass value="3.5"/>
-      <inertia ixx="0.024" ixy="0" ixz="0" iyy="0.024" iyz="0" izz="0.048"/>
-    </inertial>
-  </link>
-  <joint name="joint_fl" type="continuous">
-    <parent link="base_link"/>
-    <child link="wheel_fl"/>
-    <origin xyz="0.4 0.58 -0.24" rpy="-1.5708 0 0"/>
-    <axis xyz="0 0 1"/>
-    <dynamics damping="0.1" friction="0.5"/>
-  </joint>
-  <!-- Sol arka tekerlek -->
-  <link name="wheel_rl">
-    <inertial>
-      <mass value="3.5"/>
-      <inertia ixx="0.024" ixy="0" ixz="0" iyy="0.024" iyz="0" izz="0.048"/>
-    </inertial>
-  </link>
-  <joint name="joint_rl" type="continuous">
-    <parent link="base_link"/>
-    <child link="wheel_rl"/>
-    <origin xyz="-0.4 0.58 -0.24" rpy="-1.5708 0 0"/>
-    <axis xyz="0 0 1"/>
-    <dynamics damping="0.1" friction="0.5"/>
-  </joint>
-  <!-- Sağ ön tekerlek -->
-  <link name="wheel_fr">
-    <inertial>
-      <mass value="3.5"/>
-      <inertia ixx="0.024" ixy="0" ixz="0" iyy="0.024" iyz="0" izz="0.048"/>
-    </inertial>
-  </link>
-  <joint name="joint_fr" type="continuous">
-    <parent link="base_link"/>
-    <child link="wheel_fr"/>
-    <origin xyz="0.4 -0.58 -0.24" rpy="-1.5708 0 0"/>
-    <axis xyz="0 0 1"/>
-    <dynamics damping="0.1" friction="0.5"/>
-  </joint>
-  <!-- Sağ arka tekerlek -->
-  <link name="wheel_rr">
-    <inertial>
-      <mass value="3.5"/>
-      <inertia ixx="0.024" ixy="0" ixz="0" iyy="0.024" iyz="0" izz="0.048"/>
-    </inertial>
-  </link>
-  <joint name="joint_rr" type="continuous">
-    <parent link="base_link"/>
-    <child link="wheel_rr"/>
-    <origin xyz="-0.4 -0.58 -0.24" rpy="-1.5708 0 0"/>
-    <axis xyz="0 0 1"/>
-    <dynamics damping="0.1" friction="0.5"/>
-  </joint>
-  <!-- ─── LİDAR (RPLIDAR S2) ───────────────────── -->
+  <!-- ─── TEKERLEKLER (collision eklendi) ──────── -->
+  <xacro:macro name="tekerlek" params="isim x y">
+    <link name="${isim}">
+      <visual>
+        <origin xyz="0 0 0" rpy="0 0 0"/>
+        <geometry>
+          <cylinder radius="0.165" length="0.12"/>
+        </geometry>
+        <material name="black"><color rgba="0.1 0.1 0.1 1"/></material>
+      </visual>
+      <collision>
+        <origin xyz="0 0 0" rpy="0 0 0"/>
+        <geometry>
+          <cylinder radius="0.165" length="0.12"/>
+        </geometry>
+      </collision>
+      <inertial>
+        <mass value="3.5"/>
+        <inertia ixx="0.024" ixy="0" ixz="0" iyy="0.024" iyz="0" izz="0.048"/>
+      </inertial>
+    </link>
+    <joint name="joint_${isim}" type="continuous">
+      <parent link="base_link"/>
+      <child link="${isim}"/>
+      <!-- z=0: tekerlek merkezi base_link ile ayni hizada (zeminden 0.165m) -->
+      <origin xyz="${x} ${y} 0" rpy="-1.5708 0 0"/>
+      <axis xyz="0 0 1"/>
+      <dynamics damping="0.1" friction="0.5"/>
+    </joint>
+  </xacro:macro>
+  <xacro:tekerlek isim="wheel_fl" x="0.4"  y="0.52"/>
+  <xacro:tekerlek isim="wheel_rl" x="-0.4" y="0.52"/>
+  <xacro:tekerlek isim="wheel_fr" x="0.4"  y="-0.52"/>
+  <xacro:tekerlek isim="wheel_rr" x="-0.4" y="-0.52"/>
+  <!-- ─── LİDAR ─────────────────────────────────── -->
   <link name="lidar_link">
     <visual>
       <geometry><cylinder radius="0.04" length="0.04"/></geometry>
-      <material name="black"><color rgba="0 0 0 1"/></material>
+      <material name="lidar_black"><color rgba="0 0 0 1"/></material>
     </visual>
     <inertial>
@@ -120,6 +90,5 @@
     <parent link="base_link"/>
     <child link="lidar_link"/>
-    <!-- Şasi üstü ortasına monte -->
-    <origin xyz="0.3 0 0.14" rpy="0 0 0"/>
+    <origin xyz="0.3 0 0.4" rpy="0 0 0"/>
   </joint>
   <!-- ─── REALSENSE D455 ────────────────────────── -->
@@ -127,5 +96,5 @@
     <visual>
       <geometry><box size="0.09 0.025 0.025"/></geometry>
-      <material name="blue"><color rgba="0.0 0.2 0.8 1"/></material>
+      <material name="cam_blue"><color rgba="0.0 0.2 0.8 1"/></material>
     </visual>
     <inertial>
@@ -137,21 +106,22 @@
     <parent link="base_link"/>
     <child link="camera_link"/>
-    <!-- Ön yüze monte -->
-    <origin xyz="0.62 0 0.05" rpy="0 0 0"/>
+    <origin xyz="0.62 0 0.2" rpy="0 0 0"/>
   </joint>
   <!-- ═══════════════════════════════════════════════
        GAZEBO PLUGIN'LERİ
        ═══════════════════════════════════════════════ -->
-  <!-- Diff Drive (Skid Steer) -->
+  <gazebo>
+    <plugin filename="gz-sim-joint-state-publisher-system"
+            name="gz::sim::systems::JointStatePublisher">
+      <topic>/joint_states</topic>
+    </plugin>
+  </gazebo>
   <gazebo>
     <plugin filename="gz-sim-diff-drive-system"
             name="gz::sim::systems::DiffDrive">
-      <!-- Sol tekerlekler -->
-      <left_joint>joint_fl</left_joint>
-      <left_joint>joint_rl</left_joint>
-      <!-- Sağ tekerlekler -->
-      <right_joint>joint_fr</right_joint>
-      <right_joint>joint_rr</right_joint>
-      <!-- Elektrik ekibi hesapları -->
+      <left_joint>joint_wheel_fl</left_joint>
+      <left_joint>joint_wheel_rl</left_joint>
+      <right_joint>joint_wheel_fr</right_joint>
+      <right_joint>joint_wheel_rr</right_joint>
       <wheel_separation>1.04</wheel_separation>
       <wheel_radius>0.165</wheel_radius>
@@ -160,6 +130,6 @@
       <max_wheel_torque>21.6</max_wheel_torque>
       <max_linear_acceleration>5.0</max_linear_acceleration>
-      <topic>cmd_vel</topic>
-      <odom_topic>odom</odom_topic>
+      <topic>/cmd_vel</topic>
+      <odom_topic>/odom</odom_topic>
       <frame_id>odom</frame_id>
       <child_frame_id>base_footprint</child_frame_id>
@@ -167,5 +137,4 @@
     </plugin>
   </gazebo>
-  <!-- LiDAR (RPLIDAR S2) -->
   <gazebo reference="lidar_link">
     <sensor name="rplidar_s2" type="gpu_lidar">
@@ -187,13 +156,7 @@
           <resolution>0.03</resolution>
         </range>
-        <noise>
-          <type>gaussian</type>
-          <mean>0.0</mean>
-          <stddev>0.03</stddev>
-        </noise>
       </lidar>
     </sensor>
   </gazebo>
-  <!-- RealSense D455 Derinlik Kamerası -->
   <gazebo reference="camera_link">
     <sensor name="realsense_d455" type="depth_camera">
@@ -212,27 +175,21 @@
           <far>6.0</far>
         </clip>
-        <noise>
-          <type>gaussian</type>
-          <mean>0.0</mean>
-          <stddev>0.005</stddev>
-        </noise>
       </camera>
     </sensor>
   </gazebo>
-  <!-- Tekerlek sürtünme katsayıları -->
   <gazebo reference="wheel_fl">
-    <mu1>0.8</mu1><mu2>0.8</mu2>
+    <mu1>1.0</mu1><mu2>1.0</mu2>
     <kp>1000000.0</kp><kd>1.0</kd>
   </gazebo>
   <gazebo reference="wheel_rl">
-    <mu1>0.8</mu1><mu2>0.8</mu2>
+    <mu1>1.0</mu1><mu2>1.0</mu2>
     <kp>1000000.0</kp><kd>1.0</kd>
   </gazebo>
   <gazebo reference="wheel_fr">
-    <mu1>0.8</mu1><mu2>0.8</mu2>
+    <mu1>1.0</mu1><mu2>1.0</mu2>
     <kp>1000000.0</kp><kd>1.0</kd>
   </gazebo>
   <gazebo reference="wheel_rr">
-    <mu1>0.8</mu1><mu2>0.8</mu2>
+    <mu1>1.0</mu1><mu2>1.0</mu2>
     <kp>1000000.0</kp><kd>1.0</kd>
   </gazebo>

Commit message: S-01 parkur duzeltmeleri: basamakli rampa, engel mesafeleri arttirildi
- s01_robotlu_world.sdf: Egimli kutu rampa yerine 10 basamakli merdiven
  rampa (4.5cm adim yuksekligi, 45cm toplam), 1.5m duz tepe platformu,
  gövde collision kutusu 1.316m->0.85m (tekerlek onculugu), yan_egim
  x=7->9m, blok_15cm x=11->12m, tum engellere mu=2.0 surtuenme,
  max_wheel_torque=50Nm, ODE fizik cozucu eklendi
- urdf/robot.urdf.xacro: Arac gorunumu duzeltildi (STL mirror +90 derece)
- e02_duz_world.sdf, s02_hedef_world.sdf: Arac mesh ve collision guncellendi
- s01_tam_parkur_testi.py: fren_yapildi flag (sonsuz dongu duzeltildi),
  engel bolgeleri ve timeout guncellendi

Co-Authored-By: Claude Sonnet 4.6 <noreply@anthropic.com>

File: urdf/robot.urdf.xacro (robot description, xacro)
@@ -28,5 +28,5 @@
     </visual>
     <collision>
-      <origin xyz="0 0 0.1425" rpy="0 0 0"/>
+      <origin xyz="0 0 0.1925" rpy="0 0 0"/>
       <geometry>
         <box size="1.316 1.207 0.615"/>

Commit message: sync: Zehra'nin govde mesh (tulpar_govde_final) + urdf guncellemesi alindi
Zehra'nin feature/zehra-slalom-core (83d9f6a) commit'inden urdf/robot.urdf.xacro
ve meshes/tulpar_govde_final.stl dosyalari aynen alindi.

Not: tulpar_govde_final.stl, MD5 karsilastirmasiyla dogrulandi - onceden
kullandigimiz tulpar_ika_assembly.stl ile bayt-bayt ozdes (ayni test cubugu
ve gomulu tekerlek geometrisini iceriyor, temizlenmemis). Tekerlek yaricapi/
kutle (0.166/64kg -> 0.20/65kg) ve kamera cozunurlugu/update_rate (640x480
-> 320x240) da onceki degerlerine dondu. Bunlar kullaniciya bildirildi,
yine de Zehra'nin talimati harfiyen uygulanmasi istendi.

Co-Authored-By: Claude Sonnet 5 <noreply@anthropic.com>

File: urdf/robot.urdf.xacro (robot description, xacro)
@@ -17,32 +17,24 @@
     <parent link="base_footprint"/>
     <child link="base_link"/>
-    <!-- z=0.166: gercek tekerlek yaricapi (govde mesh'inden - tulpar_ika_assembly.stl
-         icindeki gomulu eski tekerlek geometrisinin olcumu, bkz. "cifte tekerlek"
-         notu - 0.200 degeri Zehra'nin dogrulanmamis DiffDrive degeriydi, govde
-         ile orantisiz gorunuyordu, 17 Temmuz'da duzeltildi) -->
-    <origin xyz="0 0 0.166" rpy="0 0 0"/>
+    <origin xyz="0 0 0.200" rpy="0 0 0"/>
   </joint>
   <link name="base_link">
     <visual>
-      <origin xyz="0.600 -0.300 0.110" rpy="0 0 1.5708"/>
-      <geometry>
-        <mesh filename="package://tulpar_description/meshes/tulpar_ika_assembly_tekersiz.stl" scale="0.001 0.001 0.001"/>
+      <origin xyz="0.592 -0.225 0.110" rpy="0 0 1.5708"/>
+      <geometry>
+        <mesh filename="package://tulpar_description/meshes/tulpar_govde_final.stl" scale="0.001 0.001 0.001"/>
       </geometry>
       <material name="aluminium"/>
     </visual>
     <collision>
-      <!-- z=0.187: gercek (transform uygulanmis) mesh bbox merkezinden turetilen
-           deger, ADIM2/URDF v3.0 calismasindan korunuyor -->
-      <origin xyz="0 0 0.187" rpy="0 0 0"/>
-      <geometry>
-        <box size="1.200 0.450 0.245"/>
+      <origin xyz="0 0 0.1925" rpy="0 0 0"/>
+      <geometry>
+        <box size="1.150 1.207 0.615"/>
       </geometry>
     </collision>
     <inertial>
-      <mass value="64.0"/>
+      <mass value="65.0"/>
       <origin xyz="0 0 0" rpy="0 0 0"/>
-      <!-- Analitik kutu (1.2x0.45x0.245m, 64.0kg) - fiziksel olarak garantili
-           gecerli (ucgen esitsizligi tam saglaniyor) -->
-      <inertia ixx="1.4001" ixy="0.0" ixz="0.0" iyy="8.0001" iyz="0.0" izz="8.7600"/>
+      <inertia ixx="9.94" ixy="0.0" ixz="0.0" iyy="9.21" iyz="0.0" izz="15.06"/>
     </inertial>
   </link>
@@ -50,17 +42,17 @@
     <link name="${name}">
       <visual>
-        <geometry>
-          <cylinder radius="0.166" length="0.12"/>
-        </geometry>
-        <material name="black"/>
-      </visual>
+    <geometry>
+      <cylinder radius="0.10" length="0.125"/>
+    </geometry>
+    <material name="aluminium"/>
+  </visual>
       <collision>
         <geometry>
-          <cylinder radius="0.166" length="0.12"/>
+          <cylinder radius="0.20" length="0.12"/>
         </geometry>
       </collision>
       <inertial>
         <mass value="3.5"/>
-        <inertia ixx="0.024" ixy="0" ixz="0" iyy="0.024" iyz="0" izz="0.048"/>
+        <inertia ixx="0.039" ixy="0" ixz="0" iyy="0.039" iyz="0" izz="0.070"/>
       </inertial>
     </link>
@@ -73,8 +65,8 @@
     </joint>
   </xacro:macro>
-  <xacro:wheel name="wheel_fl" x="0.39" y="0.53"/>
-  <xacro:wheel name="wheel_rl" x="-0.39" y="0.53"/>
-  <xacro:wheel name="wheel_fr" x="0.39" y="-0.53"/>
-  <xacro:wheel name="wheel_rr" x="-0.39" y="-0.53"/>
+  <xacro:wheel name="wheel_fl" x="0.4" y="0.58"/>
+  <xacro:wheel name="wheel_rl" x="-0.4" y="0.58"/>
+  <xacro:wheel name="wheel_fr" x="0.4" y="-0.58"/>
+  <xacro:wheel name="wheel_rr" x="-0.4" y="-0.58"/>
   <link name="lidar_link">
     <visual>
@@ -100,4 +92,5 @@
     <origin xyz="0 0 0" rpy="0 0 0"/>
   </joint>
+  <!-- Intel RealSense D435if depth camera. -->
   <link name="d435if_link">
     <visual>
@@ -141,6 +134,8 @@
     <origin xyz="0 0 0" rpy="-1.5708 0 -1.5708"/>
   </joint>
+  <!-- Raspberry Pi HQ camera with 16 mm telephoto lens (atis kamerasi). -->
   <link name="rpi_hq_camera_link">
     <visual>
+      <origin xyz="-0.008 0 0" rpy="0 0 0"/>
       <geometry>
         <box size="0.038 0.038 0.018"/>
@@ -148,7 +143,14 @@
       <material name="sensor_gray"/>
     </visual>
-    <inertial>
-      <mass value="0.05"/>
-      <inertia ixx="0.0004" ixy="0" ixz="0" iyy="0.0004" iyz="0" izz="0.0004"/>
+    <visual>
+      <origin xyz="0.020 0 0" rpy="0 1.5708 0"/>
+      <geometry>
+        <cylinder radius="0.018" length="0.040"/>
+      </geometry>
+      <material name="black"/>
+    </visual>
+    <inertial>
+      <mass value="0.09"/>
+      <inertia ixx="0.0008" ixy="0" ixz="0" iyy="0.0008" iyz="0" izz="0.0005"/>
     </inertial>
   </link>
@@ -164,14 +166,15 @@
     <origin xyz="0 0 0" rpy="-1.5708 0 -1.5708"/>
   </joint>
+  <!-- Rear camera: SJCAM SJ4000 action camera. -->
   <link name="rear_camera_link">
     <visual>
       <geometry>
-        <box size="0.06 0.03 0.03"/>
+        <box size="0.059 0.041 0.029"/>
       </geometry>
       <material name="sensor_gray"/>
     </visual>
     <inertial>
-      <mass value="0.07"/>
-      <inertia ixx="0.0008" ixy="0" ixz="0" iyy="0.0008" iyz="0" izz="0.0008"/>
+      <mass value="0.058"/>
+      <inertia ixx="0.0006" ixy="0" ixz="0" iyy="0.0006" iyz="0" izz="0.0006"/>
     </inertial>
   </link>
@@ -198,6 +201,6 @@
       <right_joint>joint_wheel_fr</right_joint>
       <right_joint>joint_wheel_rr</right_joint>
-      <wheel_separation>1.06</wheel_separation>
-      <wheel_radius>0.166</wheel_radius>
+      <wheel_separation>1.16</wheel_separation>
+      <wheel_radius>0.20</wheel_radius>
       <max_linear_velocity>1.0</max_linear_velocity>
       <max_angular_velocity>3.0</max_angular_velocity>
@@ -213,10 +216,10 @@
   <gazebo reference="lidar_link">
     <sensor name="ydlidar_tg30" type="gpu_lidar">
-      <update_rate>5</update_rate>
+     <update_rate>2</update_rate>
       <topic>/scan</topic>
       <lidar>
         <scan>
           <horizontal>
-            <samples>720</samples>
+            <samples>360</samples>
             <resolution>1</resolution>
             <min_angle>-3.14159</min_angle>
@@ -236,11 +239,11 @@
   <gazebo reference="d435if_link">
     <sensor name="d435if_depth" type="depth_camera">
-      <update_rate>10</update_rate>
+    <update_rate>2</update_rate>
       <topic>/d435if/depth/image_raw</topic>
       <camera>
         <horizontal_fov>1.5184</horizontal_fov>
-        <image>
-          <width>640</width>
-          <height>480</height>
+       <image>
+      <width>320</width>
+      <height>240</height>
           <format>R8G8B8</format>
         </image>
@@ -256,11 +259,11 @@
   <gazebo reference="rpi_hq_camera_link">
     <sensor name="rpi_hq_camera" type="camera">
-      <update_rate>10</update_rate>
+      <update_rate>1</update_rate>
       <topic>/rpi_hq_camera/image_raw</topic>
       <camera>
         <horizontal_fov>0.6606</horizontal_fov>
         <image>
-          <width>640</width>
-          <height>480</height>
+          <width>320</width>
+  <height>240</height>
           <format>R8G8B8</format>
         </image>
@@ -276,11 +279,11 @@
   <gazebo reference="rear_camera_link">
     <sensor name="rear_camera" type="camera">
-      <update_rate>5</update_rate>
+      <update_rate>1</update_rate>
       <topic>/rear_camera/image_raw</topic>
       <camera>
         <horizontal_fov>1.5708</horizontal_fov>
         <image>
-          <width>640</width>
-          <height>480</height>
+          <width>320</width>
+          <height>240</height>
           <format>R8G8B8</format>
         </image>
