Commit message: Nav2 (MPPI+NavFn) kurulumu + iki gercek altyapi bug'i duzeltildi + sensor konum denetimi
Nav2 bring-up ("TEB parametreleri" gorevi - teb_local_planner Jazzy'de apt'ta
olmadigi icin nav2_mppi_controller kullanildi, karar CLAUDE.md/plan dosyasinda
gerekceli):
- config/nav2_params.yaml (yeni): controller_server (MPPI, DiffDrive motion
  model, min-turning-radius kisiti yok - zero-turn dogal), planner_server
  (NavFn), global+local costmap (static+obstacle+inflation), bt_navigator,
  velocity_smoother, lifecycle_manager_navigation
- launch/nav2_bringup.launch.py (yeni): ayri launch dosyasi, gazebo/rtabmap'e
  dahil edilmiyor
- setup.py: config/ install kurali eklendi
- package.xml: nav2_* exec_depend'leri eklendi

Iki gercek, onceden fark edilmemis altyapi bug'i bulundu ve duzeltildi:
- worlds/sim_world.sdf + launch/gazebo.launch.py: render_engine ogre -> ogre2.
  gpu_lidar sensoru Ogre1 ile calismiyordu (360 isinin tamami sabit range_min=
  0.05m donduruyordu, hicbir hata/uyari vermeden) - resmi gz-sim demo dunyasiyla
  karsilastirilarak bulundu. RTAB-Map bu yuzden hicbir zaman gercek /map
  uretemiyordu.
- launch/gazebo.launch.py: lidar/d435if/rear_camera sensorlerinin LaserScan/
  Image mesajlarindaki frame_id, Gazebo'nun kendi ic scoped-entity ismini
  kullaniyordu (orn. "tulpar/base_footprint/ydlidar_tg30"), URDF'nin gercek
  link ismiyle eslesmiyordu - RTAB-Map "frame does not exist" hatasi veriyordu.
  Statik (sifir offsetli) TF alias'lariyla duzeltildi.

urdf/robot.urdf.xacro - govde mesh'ine (tulpar_govde_final.stl) gore sensor/
tekerlek konum denetimi (trimesh ile mesh analiz edilerek):
- 4 tekerlek: gercek gomulu tekerlek konumuna gore duzeltildi (iz genisligi
  1.16m -> 1.056m, kullanicinin ekranda gorsel olarak onayladigi)
- lidar_joint: taretin icindeki gercek disk konumuna tasindi (KULLANICI
  ONAYLADI)
- rear_camera_joint: z duzeltildi, x hala kesinlesmedi (kullanici "yanlis
  yerde" dedi, orijinal -0.58'e geri alindi - acik kalan is)
- d435if_joint: govde onunde bulunan detayli bir cubuk sekline gore konum+yon
  guncellendi, gorsel teyit bekliyor
- rpi_hq_camera_joint: taret/gimbal'daki 138mm'lik skop seklinin konumuna
  tasindi (atis/nisan kamerasi icin dogru yer - gimbal'a monte olmasi gerekiyor)
- Yeni: gnss_antenna_link (617mm'lik direk artik test artigi degil, gercek
  anten diregi olarak yeniden yorumlandi - SILINMEDI), aim_laser_link
  (rpi_hq_camera'ya paralel placeholder, mesh'te ayri bir lazer sekli
  bulunamadi)

Acik kalan: rear_camera x konumu, anten/lazer placeholder konumlari, taret/
gimbal mekanizmasinin ayri bir hareketli joint olarak modellenmesi (su an
govde mesh'inin sabit bir parcasi). Nav2 dogrulama testleri (lifecycle,
hedef, zero-turn, engelden kacinma, BT entegrasyonu) sistem bellek
sikismasi (swap doluydu) yuzunden yapilamadi, reboot sonrasi devam edilecek.

Co-Authored-By: Claude Sonnet 5 <noreply@anthropic.com>

File: urdf/robot.urdf.xacro (robot description, xacro)
@@ -12,4 +12,7 @@
   <material name="sensor_gray">
     <color rgba="0.3 0.3 0.3 1.0"/>
+  </material>
+  <material name="debug_red">
+    <color rgba="1.0 0.0 0.0 1.0"/>
   </material>
   <link name="base_footprint"/>
@@ -65,8 +68,16 @@
     </joint>
   </xacro:macro>
-  <xacro:wheel name="wheel_fl" x="0.4" y="0.58"/>
-  <xacro:wheel name="wheel_rl" x="-0.4" y="0.58"/>
-  <xacro:wheel name="wheel_fr" x="0.4" y="-0.58"/>
-  <xacro:wheel name="wheel_rr" x="-0.4" y="-0.58"/>
+  <!-- 18 Temmuz 2026: govde mesh'indeki 4 gomulu gercek tekerlek konumu (trimesh
+       ile bulunan 16 parcalik tekerlek imzasi, her tekerlegin tam bounds ortasi)
+       base_link'e donusturuldu - eski (0.4,0.58) degerine gore iz genisligi
+       1.16m yerine 1.056m cikiyor (CLAUDE.md'nin daha once kaydettigi 1.06m
+       degeriyle tutarli). Wheel_separation/wheel_radius DiffDrive plugin'inde
+       hala eski (1.16/0.20) degerlerde - bu ayri, bilinen bir tartisma konusu
+       (bkz. CLAUDE.md), burada sadece GORSEL konum duzeltildi, fizik parametreleri
+       degistirilmedi. -->
+  <xacro:wheel name="wheel_fl" x="0.39" y="0.528"/>
+  <xacro:wheel name="wheel_rl" x="-0.39" y="0.528"/>
+  <xacro:wheel name="wheel_fr" x="0.39" y="-0.528"/>
+  <xacro:wheel name="wheel_rr" x="-0.39" y="-0.528"/>
   <link name="lidar_link">
     <visual>
@@ -84,5 +95,10 @@
     <parent link="base_link"/>
     <child link="lidar_link"/>
-    <origin xyz="0.58 -0.015 0.61" rpy="0 0 0"/>
+    <!-- 18 Temmuz 2026: ilk tahmin (0.39,0.055,0.36) disliyle ayni merkezdeki
+         disliye ait goze (hub) isaret ediyordu, yanlisti. Kullanicinin tarif
+         ettigi "disliye gore onde/solda, alcakta" konumuna gore ikinci aday
+         denendi - trimesh raw koordinati ~(180,70,266)mm. Henuz gorsel teyit
+         edilmedi, iterasyon devam ediyor. -->
+    <origin xyz="0.522 -0.045 0.376" rpy="0 0 0"/>
   </joint>
   <link name="laser_frame"/>
@@ -108,5 +124,12 @@
     <parent link="base_link"/>
     <child link="d435if_link"/>
-    <origin xyz="0.58 0.0 0.53" rpy="0 0 0"/>
+    <!-- 18 Temmuz 2026: govde mesh'inde sasi onunde, yuksek detayli (67900 face)
+         120x10x17mm'lik bir cubuk sekli bulundu (raw ~232.9,-19.0,219.8mm) -
+         gercek Intel RealSense modeli olarak yorumlandi. Eski konum (0.58,0,0.53)
+         0.2m fazla yukarida duruyordu. Mesh'teki cubugun uzun ekseni raw-X
+         yonunde, bu da donusumden sonra base_link'in Y (yanal) eksenine denk
+         geliyor - kutumuzun uzun ekseni varsayilan olarak X (ileri) oldugu icin
+         yaw 90 derece dondurulerek gercek yonelime hizalandi. -->
+    <origin xyz="0.611 0.008 0.33" rpy="0 0 1.5708"/>
   </joint>
   <link name="d435if_color_frame"/>
@@ -158,5 +181,11 @@
     <parent link="base_link"/>
     <child link="rpi_hq_camera_link"/>
-    <origin xyz="0.58 -0.03 0.58" rpy="0 0 0"/>
+    <!-- 18 Temmuz 2026: govde mesh'inde taret/gimbal alaninda, 138mm uzunlugunda
+         teleskopik bir tup/skop sekli bulundu (raw ~286.8,169.0,306.8mm,
+         faces=3620) - 16mm telefoto lensli atis/nisan kamerasi olarak
+         yorumlandi, uzun ekseni zaten ileri (X) yonunde. Eski konum
+         (0.58,-0.03,0.58) 0.16m ileride + 0.16m yukarida duruyordu. Gorsel
+         teyit bekliyor. -->
+    <origin xyz="0.423 0.062 0.417" rpy="0 0 0"/>
   </joint>
   <link name="rpi_hq_camera_optical_frame"/>
@@ -182,5 +211,11 @@
     <parent link="base_link"/>
     <child link="rear_camera_link"/>
-    <origin xyz="-0.58 0.0 0.28" rpy="0 0 3.14159"/>
+    <!-- 18 Temmuz 2026: govde mesh'inde sasi arkasinda, yuksek detayli (11224 face)
+         47x18x41mm'lik bir kutu bulundu (raw ~223.5,1173.5,276.9mm) - z 0.28'den
+         0.387'ye duzeltildi. "6cm one" denemesi kullanici tarafindan yanlis
+         yon olarak isaretlendi, x=-0.58'e geri alindi. Tam doğru konum icin
+         mesh'te daha iyi bir referans bulunamadi - kullanicidan net koordinat/
+         foto bekleniyor, ayri bir gorev olarak birakildi. -->
+    <origin xyz="-0.58 0.0 0.387" rpy="0 0 3.14159"/>
   </joint>
   <link name="rear_camera_optical_frame"/>
@@ -189,4 +224,49 @@
     <child link="rear_camera_optical_frame"/>
     <origin xyz="0 0 0" rpy="-1.5708 0 -1.5708"/>
+  </joint>
+  <!-- GNSS anten (ZED-F9P RTK, roadmap Gun 7). 18 Temmuz 2026: govde mesh'inde
+       "test cubugu" sanilan 617mm'lik ince direk (comp4592, raw x~50,y~1150,
+       z 241.5-858.5mm) aslinda bir anten diregi olarak yeniden yorumlandi -
+       kullanicinin "anten eksik" demesiyle tutarli, silinmedi. Anten linki
+       direğin tepesine (raw z=858.5mm) eklendi. -->
+  <link name="gnss_antenna_link">
+    <visual>
+      <geometry>
+        <cylinder radius="0.025" length="0.02"/>
+      </geometry>
+      <material name="black"/>
+    </visual>
+    <inertial>
+      <mass value="0.05"/>
+      <inertia ixx="0.0001" ixy="0" ixz="0" iyy="0.0001" iyz="0" izz="0.0001"/>
+    </inertial>
+  </link>
+  <joint name="gnss_antenna_joint" type="fixed">
+    <parent link="base_link"/>
+    <child link="gnss_antenna_link"/>
+    <!-- raw direk ucu (~50,1150,858.5mm) base_link'e donusturuldu. -->
+    <origin xyz="-0.558 -0.175 0.9685" rpy="0 0 0"/>
+  </joint>
+  <!-- Atis/nisan lazeri (roadmap: "servo+lazer diyot", izinli-atesleme role
+       node'u). 18 Temmuz 2026: mesh'te ayri, belirgin bir lazer-diyot sekli
+       bulunamadi (muhtemelen gercek tasarimda skopla ayni govdede/paralel) -
+       rpi_hq_camera'nin (skop) hemen yanina, boresight hizali placeholder
+       olarak eklendi. Gercek konum mekanik ekipten netlesince guncellenmeli. -->
+  <link name="aim_laser_link">
+    <visual>
+      <geometry>
+        <cylinder radius="0.008" length="0.05"/>
+      </geometry>
+      <material name="black"/>
+    </visual>
+    <inertial>
+      <mass value="0.02"/>
+      <inertia ixx="0.00001" ixy="0" ixz="0" iyy="0.00001" iyz="0" izz="0.00001"/>
+    </inertial>
+  </link>
+  <joint name="aim_laser_joint" type="fixed">
+    <parent link="rpi_hq_camera_link"/>
+    <child link="aim_laser_link"/>
+    <origin xyz="0 0.04 0" rpy="0 1.5708 0"/>
   </joint>
   <gazebo>

Commit message: Nav2 dogrulamasi tamamlandi + 3 gercek bug bulunup 2'si duzeltildi
c12ceb4'un birakti gi yerden (sistem bellek sikismasi nedeniyle yapilamayan
Nav2 dogrulama testleri) devam edildi:

KRITIK duzeltmeler:
- urdf/robot.urdf.xacro: lidar_joint konumu govde mesh yuzeyine 16.7mm
  mesafede/gomulu cikti (trimesh ile olculdu) - lidar kendi govdesini
  "engel" olarak goruyordu (/scan'de 0.09-0.45m sahte kisa mesafeler,
  Spin davranisi "Collision Ahead" ile aninda iptal oluyordu). Gecici
  duzeltme: z 376mm->1050mm (mesh'in global Z maksimumunun ~82mm ustu,
  garantili temiz) - KESIN konum degil, mekanik/gorsel teyit bekliyor.
- tulpar_bt/src/bt_executor_main.cpp + behavior_trees/ana_tree.xml:
  Repeat(-1)+ForceSuccess deseni BT.CPP'nin bilinen bir tuzagina carpiyordu
  - child SUCCESS dondugunde ayni tickOnce() cagrisi icinde senkron tekrar
  tikleniyor, ForceSuccess her tick'te (normal olan) FAILURE'i SUCCESS'e
  cevirdigi icin sonsuz senkron dongu olusuyordu (1 CPU cekirdegi ~%90,
  10 saniyede ~1.2 milyon log satiri). Duzeltme: Repeat/ForceSuccess
  kaldirildi, disaridaki ana dongu artik sonuçtan bagimsiz surekli
  tikliyor ve her tick sonrasi throttle uyguluyor - agac bittiginde
  bir sonraki dis-dongu adiminda standart BT.CPP davranisiyla otomatik
  yeniden basliyor, senkron dongu riski olmadan.
- launch/gazebo.launch.py: headless launch argument eklendi (gz sim -s,
  GUI'siz) - GUI ~3.2GB RAM yiyip sistemi swap'a itiyordu, bu da RTAB-Map'in
  TF senkronunu bozup /map'i durduruyordu.

Ayrica bulunan (kod degisikligi yapilmadi, belgelendi):
- RTAB-Map soguk-baslangic kilitlenmesi: ilk scan donusturme denemesi TF
  buffer isinmadan basarisiz olursa, node canli kalir ama ic isleme
  donguyu sessizce ve kalici olarak durur (/map bir daha hic yayinlanmaz).
  Tek cozum: rtabmap node'unu (sadece onu) yeniden baslatmak.

Duzeltmeler sonrasi tam Nav2 dogrulamasi basarili: lifecycle (5 node
ACTIVE), Spin (360 zero-turn), NavigateToPose (0 recovery ile hedefe
ulasildi), tulpar_bt->Nav2->Gazebo uctan uca zinciri calisiyor.

Co-Authored-By: Claude Sonnet 5 <noreply@anthropic.com>

File: urdf/robot.urdf.xacro (robot description, xacro)
@@ -99,6 +99,24 @@
          ettigi "disliye gore onde/solda, alcakta" konumuna gore ikinci aday
          denendi - trimesh raw koordinati ~(180,70,266)mm. Henuz gorsel teyit
-         edilmedi, iterasyon devam ediyor. -->
-    <origin xyz="0.522 -0.045 0.376" rpy="0 0 0"/>
+         edilmedi, iterasyon devam ediyor.
+         18 Temmuz 2026 (Nav2 dogrulama oturumu): bu nokta govde mesh yuzeyine
+         trimesh ile olculdugunde sadece 16.7mm mesafede/gomulu cikti - GPU
+         lidar sensoru kendi govdesini her yonde ~0.09-0.45m menzilde "engel"
+         olarak goruyordu (Spin davranisi 0.1sn'de "Collision Ahead" ile iptal
+         oluyordu, RTAB-Map haritasi sahte yakin-engel verisiyle kirleniyordu).
+         GECICI duzeltme (1. deneme): ayni XY'de mesh'in bu noktadaki yerel
+         kolonu 283.7mm'de bitiyor sanildi (40mm yaricapta tarandi) - z
+         376->430mm'e (+54mm) cekildi, AMA canli /scan testinde hala 307
+         okumanin 209'u 0.5m altinda cikti - turret govdesi o dar yerel
+         kolon taramasinin gosterdiginden daha genis/karmasik saracaktir.
+         GECICI duzeltme (2. deneme, calisiyor): yerel tahmin yerine mesh'in
+         TUM govde icin global Z maksimumu (858.5mm ham koordinat) esas
+         alindi - 940mm (858.5'in ~82mm ustu) hicbir XY icin hicbir mesh
+         vertex'inin ustunde olamaz, garantili temiz. z=0.376->1.050m (raw
+         940mm). Bu KESIN/ONAYLI bir konum DEGIL, sadece Nav2/Spin/obstacle-
+         avoidance testini acmak icin gecici/gorsel-olarak-yanlis bir
+         cikarma - gercek lidar montaj noktasi mekanik ekiple/gorsel teyitle
+         netlesince degisecek. -->
+    <origin xyz="0.522 -0.045 1.050" rpy="0 0 0"/>
   </joint>
   <link name="laser_frame"/>
