Commit message: Fusion CAD entegrasyonu tamamlandi + Gazebo render sorunu cozumu + IMU
- Halil'in gerçek CAD mesh'leri (lidar2_v1_1, wifi radio/anten, tulpar_ika_assembly)
  repoya eklendi - urdf/robot.urdf.xacro'da referans veriliyor ama commit
  edilmemişlerdi (Gün 7).
- Canlı-spawn edilen 149MB/~3M-yüzey gövde mesh'i Gazebo GUI'sinde tutarsız
  render sorununa yol açıyordu (Entity Tree'de görünmeme/parçalanmış görünme) -
  kök neden GPU sürücüsü değil, mesh boyutuydu (gz model -p ve /joint_states
  fizik motorunun sürekli stabil olduğunu doğruladı). Görsel-only kopyaları
  (tulpar_ika_assembly_visual.stl 565k yüzey/28MB, lidar2_v1_1_visual.stl 5k
  yüzey) trimesh.simplify_quadric_decimation ile üretildi, collision/inertia'ya
  dokunulmadı.
- IMU sensörü eklendi (Gazebo imu sensörü + gz-sim-imu-system plugin, ~97Hz) -
  önceki oturumda askıya alınan karar netleşti.
- nav2_params.yaml footprint + collision_checker_node.py robot_radius_m,
  Fusion CAD'den türetilen gerçek ölçülerle senkronlandı (0.835->0.850).

Not: Gazebo GUI'de farklı, çözülemeyen bir görsel "patlama" sorunu hâlâ açık
(fizik davranışını etkilemiyor, sadece render) - bkz. CLAUDE.md Gün 8.

Co-Authored-By: Claude Sonnet 5 <noreply@anthropic.com>

File: urdf/robot.urdf.xacro (robot description, xacro)
@@ -13,18 +13,18 @@
     <color rgba="0.3 0.3 0.3 1.0"/>
   </material>
-  <material name="debug_red">
-    <color rgba="1.0 0.0 0.0 1.0"/>
-  </material>
+  <xacro:property name="cad_center_x" value="0.225"/>
+  <xacro:property name="cad_center_y" value="0.592375"/>
+  <xacro:property name="cad_z_offset" value="0.109663086"/>
   <link name="base_footprint"/>
   <joint name="base_joint" type="fixed">
     <parent link="base_footprint"/>
     <child link="base_link"/>
-    <origin xyz="0 0 0.200" rpy="0 0 0"/>
+    <origin xyz="0 0 0.165" rpy="0 0 0"/>
   </joint>
   <link name="base_link">
     <visual>
-      <origin xyz="0.592 -0.225 0.110" rpy="0 0 1.5708"/>
-      <geometry>
-        <mesh filename="package://tulpar_description/meshes/tulpar_govde_final.stl" scale="0.001 0.001 0.001"/>
+      <origin xyz="${cad_center_y} ${-cad_center_x} ${cad_z_offset}" rpy="0 0 1.57079633"/>
+      <geometry>
+        <mesh filename="package://tulpar_description/meshes/tulpar_ika_assembly_visual.stl" scale="0.001 0.001 0.001"/>
       </geometry>
       <material name="aluminium"/>
@@ -33,5 +33,5 @@
       <origin xyz="0 0 0.1925" rpy="0 0 0"/>
       <geometry>
-        <box size="1.150 1.207 0.615"/>
+        <box size="1.1666 1.2368 0.615"/>
       </geometry>
     </collision>
@@ -45,17 +45,17 @@
     <link name="${name}">
       <visual>
-    <geometry>
-      <cylinder radius="0.10" length="0.125"/>
-    </geometry>
-    <material name="aluminium"/>
-  </visual>
+        <geometry>
+          <cylinder radius="0.165" length="0.125"/>
+        </geometry>
+        <material name="black"/>
+      </visual>
       <collision>
         <geometry>
-          <cylinder radius="0.20" length="0.12"/>
+          <cylinder radius="0.165" length="0.12"/>
         </geometry>
       </collision>
       <inertial>
         <mass value="3.5"/>
-        <inertia ixx="0.039" ixy="0" ixz="0" iyy="0.039" iyz="0" izz="0.070"/>
+        <inertia ixx="0.024" ixy="0" ixz="0" iyy="0.024" iyz="0" izz="0.048"/>
       </inertial>
     </link>
@@ -68,26 +68,18 @@
     </joint>
   </xacro:macro>
-  <!-- 18 Temmuz 2026: govde mesh'indeki 4 gomulu gercek tekerlek konumu (trimesh
-       ile bulunan 16 parcalik tekerlek imzasi, her tekerlegin tam bounds ortasi)
-       base_link'e donusturuldu - eski (0.4,0.58) degerine gore iz genisligi
-       1.16m yerine 1.056m cikiyor (CLAUDE.md'nin daha once kaydettigi 1.06m
-       degeriyle tutarli). Wheel_separation/wheel_radius DiffDrive plugin'inde
-       hala eski (1.16/0.20) degerlerde - bu ayri, bilinen bir tartisma konusu
-       (bkz. CLAUDE.md), burada sadece GORSEL konum duzeltildi, fizik parametreleri
-       degistirilmedi. -->
-  <xacro:wheel name="wheel_fl" x="0.39" y="0.528"/>
-  <xacro:wheel name="wheel_rl" x="-0.39" y="0.528"/>
-  <xacro:wheel name="wheel_fr" x="0.39" y="-0.528"/>
-  <xacro:wheel name="wheel_rr" x="-0.39" y="-0.528"/>
+  <xacro:wheel name="wheel_fl" x="0.4" y="0.52"/>
+  <xacro:wheel name="wheel_rl" x="-0.4" y="0.52"/>
+  <xacro:wheel name="wheel_fr" x="0.4" y="-0.52"/>
+  <xacro:wheel name="wheel_rr" x="-0.4" y="-0.52"/>
   <link name="lidar_link">
     <visual>
       <geometry>
-        <cylinder radius="0.05" length="0.06"/>
+        <mesh filename="package://tulpar_description/meshes/lidar2_v1_1_visual.stl"/>
       </geometry>
       <material name="sensor_gray"/>
     </visual>
     <inertial>
-      <mass value="0.25"/>
-      <inertia ixx="0.0015" ixy="0" ixz="0" iyy="0.0015" iyz="0" izz="0.0015"/>
+      <mass value="0.275"/>
+      <inertia ixx="0.00024" ixy="0" ixz="0" iyy="0.00019" iyz="0" izz="0.00034"/>
     </inertial>
   </link>
@@ -95,28 +87,5 @@
     <parent link="base_link"/>
     <child link="lidar_link"/>
-    <!-- 18 Temmuz 2026: ilk tahmin (0.39,0.055,0.36) disliyle ayni merkezdeki
-         disliye ait goze (hub) isaret ediyordu, yanlisti. Kullanicinin tarif
-         ettigi "disliye gore onde/solda, alcakta" konumuna gore ikinci aday
-         denendi - trimesh raw koordinati ~(180,70,266)mm. Henuz gorsel teyit
-         edilmedi, iterasyon devam ediyor.
-         18 Temmuz 2026 (Nav2 dogrulama oturumu): bu nokta govde mesh yuzeyine
-         trimesh ile olculdugunde sadece 16.7mm mesafede/gomulu cikti - GPU
-         lidar sensoru kendi govdesini her yonde ~0.09-0.45m menzilde "engel"
-         olarak goruyordu (Spin davranisi 0.1sn'de "Collision Ahead" ile iptal
-         oluyordu, RTAB-Map haritasi sahte yakin-engel verisiyle kirleniyordu).
-         GECICI duzeltme (1. deneme): ayni XY'de mesh'in bu noktadaki yerel
-         kolonu 283.7mm'de bitiyor sanildi (40mm yaricapta tarandi) - z
-         376->430mm'e (+54mm) cekildi, AMA canli /scan testinde hala 307
-         okumanin 209'u 0.5m altinda cikti - turret govdesi o dar yerel
-         kolon taramasinin gosterdiginden daha genis/karmasik saracaktir.
-         GECICI duzeltme (2. deneme, calisiyor): yerel tahmin yerine mesh'in
-         TUM govde icin global Z maksimumu (858.5mm ham koordinat) esas
-         alindi - 940mm (858.5'in ~82mm ustu) hicbir XY icin hicbir mesh
-         vertex'inin ustunde olamaz, garantili temiz. z=0.376->1.050m (raw
-         940mm). Bu KESIN/ONAYLI bir konum DEGIL, sadece Nav2/Spin/obstacle-
-         avoidance testini acmak icin gecici/gorsel-olarak-yanlis bir
-         cikarma - gercek lidar montaj noktasi mekanik ekiple/gorsel teyitle
-         netlesince degisecek. -->
-    <origin xyz="0.522 -0.045 1.050" rpy="0 0 0"/>
+    <origin xyz="-0.010642665 -0.64000642 0.351677956" rpy="0 0 4.71238898"/>
   </joint>
   <link name="laser_frame"/>
@@ -126,15 +95,14 @@
     <origin xyz="0 0 0" rpy="0 0 0"/>
   </joint>
-  <!-- Intel RealSense D435if depth camera. -->
   <link name="d435if_link">
     <visual>
       <geometry>
-        <box size="0.09 0.025 0.025"/>
+        <box size="0.124 0.026 0.029"/>
       </geometry>
       <material name="camera_blue"/>
     </visual>
     <inertial>
-      <mass value="0.08"/>
-      <inertia ixx="0.001" ixy="0" ixz="0" iyy="0.001" iyz="0" izz="0.001"/>
+      <mass value="0.313"/>
+      <inertia ixx="0.00018" ixy="0" ixz="0" iyy="0.00055" iyz="0" izz="0.00058"/>
     </inertial>
   </link>
@@ -142,12 +110,5 @@
     <parent link="base_link"/>
     <child link="d435if_link"/>
-    <!-- 18 Temmuz 2026: govde mesh'inde sasi onunde, yuksek detayli (67900 face)
-         120x10x17mm'lik bir cubuk sekli bulundu (raw ~232.9,-19.0,219.8mm) -
-         gercek Intel RealSense modeli olarak yorumlandi. Eski konum (0.58,0,0.53)
-         0.2m fazla yukarida duruyordu. Mesh'teki cubugun uzun ekseni raw-X
-         yonunde, bu da donusumden sonra base_link'in Y (yanal) eksenine denk
-         geliyor - kutumuzun uzun ekseni varsayilan olarak X (ileri) oldugu icin
-         yaw 90 derece dondurulerek gercek yonelime hizalandi. -->
-    <origin xyz="0.611 0.008 0.33" rpy="0 0 1.5708"/>
+    <origin xyz="0.618375 0.0075 0.329663086" rpy="-1.57079633 0 -1.57079633"/>
   </joint>
   <link name="d435if_color_frame"/>
@@ -175,5 +136,4 @@
     <origin xyz="0 0 0" rpy="-1.5708 0 -1.5708"/>
   </joint>
-  <!-- Raspberry Pi HQ camera with 16 mm telephoto lens (atis kamerasi). -->
   <link name="rpi_hq_camera_link">
     <visual>
@@ -199,11 +159,5 @@
     <parent link="base_link"/>
     <child link="rpi_hq_camera_link"/>
-    <!-- 18 Temmuz 2026: govde mesh'inde taret/gimbal alaninda, 138mm uzunlugunda
-         teleskopik bir tup/skop sekli bulundu (raw ~286.8,169.0,306.8mm,
-         faces=3620) - 16mm telefoto lensli atis/nisan kamerasi olarak
-         yorumlandi, uzun ekseni zaten ileri (X) yonunde. Eski konum
-         (0.58,-0.03,0.58) 0.16m ileride + 0.16m yukarida duruyordu. Gorsel
-         teyit bekliyor. -->
-    <origin xyz="0.423 0.062 0.417" rpy="0 0 0"/>
+    <origin xyz="0.492373 0.049000 0.424228" rpy="0 0 0"/>
   </joint>
   <link name="rpi_hq_camera_optical_frame"/>
@@ -213,5 +167,4 @@
     <origin xyz="0 0 0" rpy="-1.5708 0 -1.5708"/>
   </joint>
-  <!-- Rear camera: SJCAM SJ4000 action camera. -->
   <link name="rear_camera_link">
     <visual>
@@ -229,11 +182,5 @@
     <parent link="base_link"/>
     <child link="rear_camera_link"/>
-    <!-- 18 Temmuz 2026: govde mesh'inde sasi arkasinda, yuksek detayli (11224 face)
-         47x18x41mm'lik bir kutu bulundu (raw ~223.5,1173.5,276.9mm) - z 0.28'den
-         0.387'ye duzeltildi. "6cm one" denemesi kullanici tarafindan yanlis
-         yon olarak isaretlendi, x=-0.58'e geri alindi. Tam doğru konum icin
-         mesh'te daha iyi bir referans bulunamadi - kullanicidan net koordinat/
-         foto bekleniyor, ayri bir gorev olarak birakildi. -->
-    <origin xyz="-0.58 0.0 0.387" rpy="0 0 3.14159"/>
+    <origin xyz="-0.58687500 -0.00155476 0.38655832" rpy="0 0 3.14159"/>
   </joint>
   <link name="rear_camera_optical_frame"/>
@@ -243,52 +190,82 @@
     <origin xyz="0 0 0" rpy="-1.5708 0 -1.5708"/>
   </joint>
-  <!-- GNSS anten (ZED-F9P RTK, roadmap Gun 7). 18 Temmuz 2026: govde mesh'inde
-       "test cubugu" sanilan 617mm'lik ince direk (comp4592, raw x~50,y~1150,
-       z 241.5-858.5mm) aslinda bir anten diregi olarak yeniden yorumlandi -
-       kullanicinin "anten eksik" demesiyle tutarli, silinmedi. Anten linki
-       direğin tepesine (raw z=858.5mm) eklendi. -->
-  <link name="gnss_antenna_link">
-    <visual>
-      <geometry>
-        <cylinder radius="0.025" length="0.02"/>
+  <link name="wifi_radio_link">
+    <visual>
+      <geometry>
+        <mesh filename="package://tulpar_description/meshes/Bullet_2hp_Ubiquiti_1.stl"/>
       </geometry>
       <material name="black"/>
     </visual>
     <inertial>
-      <mass value="0.05"/>
-      <inertia ixx="0.0001" ixy="0" ixz="0" iyy="0.0001" iyz="0" izz="0.0001"/>
-    </inertial>
-  </link>
-  <joint name="gnss_antenna_joint" type="fixed">
-    <parent link="base_link"/>
-    <child link="gnss_antenna_link"/>
-    <!-- raw direk ucu (~50,1150,858.5mm) base_link'e donusturuldu. -->
-    <origin xyz="-0.558 -0.175 0.9685" rpy="0 0 0"/>
-  </joint>
-  <!-- Atis/nisan lazeri (roadmap: "servo+lazer diyot", izinli-atesleme role
-       node'u). 18 Temmuz 2026: mesh'te ayri, belirgin bir lazer-diyot sekli
-       bulunamadi (muhtemelen gercek tasarimda skopla ayni govdede/paralel) -
-       rpi_hq_camera'nin (skop) hemen yanina, boresight hizali placeholder
-       olarak eklendi. Gercek konum mekanik ekipten netlesince guncellenmeli. -->
-  <link name="aim_laser_link">
-    <visual>
-      <geometry>
-        <cylinder radius="0.008" length="0.05"/>
+      <mass value="0.213"/>
+      <inertia ixx="0.0007" ixy="0" ixz="0" iyy="0.0007" iyz="0" izz="0.00006"/>
+    </inertial>
+  </link>
+  <joint name="wifi_radio_joint" type="fixed">
+    <parent link="base_link"/>
+    <child link="wifi_radio_link"/>
+    <origin xyz="-0.55664594 -0.163840659 0.142025727" rpy="0 0.019476555 3.14159265"/>
+  </joint>
+  <link name="wifi_antenna_left_link">
+    <visual>
+      <geometry>
+        <mesh filename="package://tulpar_description/meshes/WIFI_ANTENNA_P3526_1.stl"/>
       </geometry>
       <material name="black"/>
     </visual>
     <inertial>
-      <mass value="0.02"/>
-      <inertia ixx="0.00001" ixy="0" ixz="0" iyy="0.00001" iyz="0" izz="0.00001"/>
-    </inertial>
-  </link>
-  <joint name="aim_laser_joint" type="fixed">
-    <parent link="rpi_hq_camera_link"/>
-    <child link="aim_laser_link"/>
-    <origin xyz="0 0.04 0" rpy="0 1.5708 0"/>
-  </joint>
+      <mass value="0.01"/>
+      <inertia ixx="1e-05" ixy="0" ixz="0" iyy="1e-05" iyz="0" izz="1e-05"/>
+    </inertial>
+  </link>
+  <joint name="wifi_antenna_left_joint" type="fixed">
+    <parent link="base_link"/>
+    <child link="wifi_antenna_left_link"/>
+    <origin xyz="0.236314539 0.001977871 0.166971529" rpy="0 0 0"/>
+  </joint>
+  <link name="wifi_antenna_right_link">
+    <visual>
+      <geometry>
+        <mesh filename="package://tulpar_description/meshes/WIFI_ANTENNA_P3526_2.stl"/>
+      </geometry>
+      <material name="black"/>
+    </visual>
+    <inertial>
+      <mass value="0.01"/>
+      <inertia ixx="1e-05" ixy="0" ixz="0" iyy="1e-05" iyz="0" izz="1e-05"/>
+    </inertial>
+  </link>
+  <joint name="wifi_antenna_right_joint" type="fixed">
+    <parent link="base_link"/>
+    <child link="wifi_antenna_right_link"/>
+    <origin xyz="0.305717539 0.087677871 0.166971529" rpy="0 0 3.14159265"/>
+  </joint>
+  <link name="imu_link">
+    <inertial>
+      <mass value="0.01"/>
+      <inertia ixx="1e-05" ixy="0" ixz="0" iyy="1e-05" iyz="0" izz="1e-05"/>
+    </inertial>
+  </link>
+  <joint name="imu_joint" type="fixed">
+    <parent link="base_link"/>
+    <child link="imu_link"/>
+    <origin xyz="0 0 0.1925" rpy="0 0 0"/>
+  </joint>
+  <gazebo reference="imu_link">
+    <sensor name="wt901c_imu" type="imu">
+      <update_rate>100</update_rate>
+      <topic>/imu</topic>
+      <gz_frame_id>imu_link</gz_frame_id>
+      <always_on>true</always_on>
+      <visualize>false</visualize>
+    </sensor>
+  </gazebo>
   <gazebo>
     <plugin filename="gz-sim-joint-state-publisher-system" name="gz::sim::systems::JointStatePublisher">
       <topic>/joint_states</topic>
+    </plugin>
+  </gazebo>
+  <gazebo>
+    <plugin filename="gz-sim-imu-system" name="gz::sim::systems::Imu">
     </plugin>
   </gazebo>
@@ -299,6 +276,6 @@
       <right_joint>joint_wheel_fr</right_joint>
       <right_joint>joint_wheel_rr</right_joint>
-      <wheel_separation>1.16</wheel_separation>
-      <wheel_radius>0.20</wheel_radius>
+      <wheel_separation>1.04</wheel_separation>
+      <wheel_radius>0.165</wheel_radius>
       <max_linear_velocity>1.0</max_linear_velocity>
       <max_angular_velocity>3.0</max_angular_velocity>
@@ -314,10 +291,11 @@
   <gazebo reference="lidar_link">
     <sensor name="ydlidar_tg30" type="gpu_lidar">
-     <update_rate>2</update_rate>
+      <update_rate>10</update_rate>
       <topic>/scan</topic>
+      <gz_frame_id>laser_frame</gz_frame_id>
       <lidar>
         <scan>
           <horizontal>
-            <samples>360</samples>
+            <samples>800</samples>
             <resolution>1</resolution>
             <min_angle>-3.14159</min_angle>
@@ -336,12 +314,13 @@
   </gazebo>
   <gazebo reference="d435if_link">
-    <sensor name="d435if_depth" type="depth_camera">
-    <update_rate>2</update_rate>
+    <sensor name="d455_depth" type="depth_camera">
+      <update_rate>30</update_rate>
       <topic>/d435if/depth/image_raw</topic>
+      <gz_frame_id>d435if_depth_optical_frame</gz_frame_id>
       <camera>
         <horizontal_fov>1.5184</horizontal_fov>
-       <image>
-      <width>320</width>
-      <height>240</height>
+        <image>
+          <width>848</width>
+          <height>480</height>
           <format>R8G8B8</format>
         </image>
@@ -363,5 +342,5 @@
         <image>
           <width>320</width>
-  <height>240</height>
+          <height>240</height>
           <format>R8G8B8</format>
         </image>

Commit message: KRITIK duzeltme: base_link collision box X/Y ekseni ters + yukseklik hala eskiydi
Kapsamli denetim sirasinda bulundu: Gun 7'de "base_link collision box
1.237x1.167x1.133m'ye duzeltildi" diye belgelenmisti ama gercekte:
1. X/Y eksenleri ters yazilmisti (size="1.1666 1.2368 0.615" - X=1.1666
   yaziyordu ama trimesh ile govde mesh'inin gercek donusturulmus bbox'i
   X ekseninde 1.2368, Y ekseninde 1.1666 cikiyor - nav2_params.yaml'daki
   footprint [[0.6185,0.5835],...] da bunu dogruluyor, X/Y swap kesin).
2. Yukseklik hic guncellenmemisti - hala eski/yanlis 0.615m'deydi. Duzeltme
   sadece X/Y footprint'e (nav2_params.yaml) islenmis, bu collision box'a
   hic yansimamis. Gercek yukseklik govde mesh'inin tam Z araligindan
   1.1332m (merkez z=0.4016) - eski kutu aracin ust yarisini (turret/govde
   ustu, yaklasik ust 47cm) fizik motorunda hic COLLISION olarak kapsamiyordu.

Duzeltme: size="1.2368 1.1666 1.1332", origin z=0.4016. Gazebo'da 32+ saniye
stabilite testiyle dogrulandi (gz model -p sürekli sabit).

Co-Authored-By: Claude Sonnet 5 <noreply@anthropic.com>

File: urdf/robot.urdf.xacro (robot description, xacro)
@@ -31,7 +31,15 @@
     </visual>
     <collision>
-      <origin xyz="0 0 0.1925" rpy="0 0 0"/>
-      <geometry>
-        <box size="1.1666 1.2368 0.615"/>
+      <!-- 21 Temmuz 2026: eski deger (size 1.1666 1.2368 0.615, origin_z=0.1925)
+           X/Y eksenleri ters (gercek: X=1.2368 Y=1.1666, trimesh ile govde
+           mesh'inin gercek dunyaya-donusturulmus bbox'indan hesaplandi) VE
+           yukseklik hala eski/yanlis degerdeydi (0.615 - "duzeltildi"
+           denmisti ama sadece X/Y footprint'e islenmisti, bu collision box'a
+           hic yansimamis). Gercek yukseklik 1.1332m (govde mesh'inin tam Z
+           araligindan), merkez z=0.4016 - onceki kutu aracin ust yarisini
+           (turret/govde ustu) hic kapsamiyordu. -->
+      <origin xyz="0 0 0.4016" rpy="0 0 0"/>
+      <geometry>
+        <box size="1.2368 1.1666 1.1332"/>
       </geometry>
     </collision>
