Commit message: Update sensors and add slalom core utilities

File: src/tulpar_description/urdf/robot.urdf.xacro (robot description, xacro)
@@ -42,9 +42,9 @@
     <link name="${name}">
       <visual>
-        <geometry>
-          <cylinder radius="0.165" length="0.12"/>
-        </geometry>
-        <material name="black"/>
-      </visual>
+    <geometry>
+      <cylinder radius="0.10" length="0.125"/>
+    </geometry>
+    <material name="aluminium"/>
+  </visual>
       <collision>
         <geometry>
@@ -92,5 +92,6 @@
     <origin xyz="0 0 0" rpy="0 0 0"/>
   </joint>
-  <link name="d435i_link">
+  <!-- Intel RealSense D435if depth camera. -->
+  <link name="d435if_link">
     <visual>
       <geometry>
@@ -104,35 +105,37 @@
     </inertial>
   </link>
-  <joint name="d435i_joint" type="fixed">
+  <joint name="d435if_joint" type="fixed">
     <parent link="base_link"/>
-    <child link="d435i_link"/>
+    <child link="d435if_link"/>
     <origin xyz="0.62 0.0 0.20" rpy="0 0 0"/>
   </joint>
-  <link name="d435i_color_frame"/>
-  <joint name="d435i_color_joint" type="fixed">
-    <parent link="d435i_link"/>
-    <child link="d435i_color_frame"/>
+  <link name="d435if_color_frame"/>
+  <joint name="d435if_color_joint" type="fixed">
+    <parent link="d435if_link"/>
+    <child link="d435if_color_frame"/>
     <origin xyz="0 0 0" rpy="0 0 0"/>
   </joint>
-  <link name="d435i_color_optical_frame"/>
-  <joint name="d435i_color_optical_joint" type="fixed">
-    <parent link="d435i_color_frame"/>
-    <child link="d435i_color_optical_frame"/>
+  <link name="d435if_color_optical_frame"/>
+  <joint name="d435if_color_optical_joint" type="fixed">
+    <parent link="d435if_color_frame"/>
+    <child link="d435if_color_optical_frame"/>
     <origin xyz="0 0 0" rpy="-1.5708 0 -1.5708"/>
   </joint>
-  <link name="d435i_depth_frame"/>
-  <joint name="d435i_depth_joint" type="fixed">
-    <parent link="d435i_link"/>
-    <child link="d435i_depth_frame"/>
+  <link name="d435if_depth_frame"/>
+  <joint name="d435if_depth_joint" type="fixed">
+    <parent link="d435if_link"/>
+    <child link="d435if_depth_frame"/>
     <origin xyz="0 0 0" rpy="0 0 0"/>
   </joint>
-  <link name="d435i_depth_optical_frame"/>
-  <joint name="d435i_depth_optical_joint" type="fixed">
-    <parent link="d435i_depth_frame"/>
-    <child link="d435i_depth_optical_frame"/>
+  <link name="d435if_depth_optical_frame"/>
+  <joint name="d435if_depth_optical_joint" type="fixed">
+    <parent link="d435if_depth_frame"/>
+    <child link="d435if_depth_optical_frame"/>
     <origin xyz="0 0 0" rpy="-1.5708 0 -1.5708"/>
   </joint>
+  <!-- Raspberry Pi HQ camera with 16 mm telephoto lens (atis kamerasi). -->
   <link name="rpi_hq_camera_link">
     <visual>
+      <origin xyz="-0.008 0 0" rpy="0 0 0"/>
       <geometry>
         <box size="0.038 0.038 0.018"/>
@@ -140,7 +143,14 @@
       <material name="sensor_gray"/>
     </visual>
-    <inertial>
-      <mass value="0.05"/>
-      <inertia ixx="0.0004" ixy="0" ixz="0" iyy="0.0004" iyz="0" izz="0.0004"/>
+    <visual>
+      <origin xyz="0.020 0 0" rpy="0 1.5708 0"/>
+      <geometry>
+        <cylinder radius="0.018" length="0.040"/>
+      </geometry>
+      <material name="black"/>
+    </visual>
+    <inertial>
+      <mass value="0.09"/>
+      <inertia ixx="0.0008" ixy="0" ixz="0" iyy="0.0008" iyz="0" izz="0.0005"/>
     </inertial>
   </link>
@@ -156,14 +166,15 @@
     <origin xyz="0 0 0" rpy="-1.5708 0 -1.5708"/>
   </joint>
+  <!-- Rear camera: SJCAM SJ4000 action camera. -->
   <link name="rear_camera_link">
     <visual>
       <geometry>
-        <box size="0.06 0.03 0.03"/>
+        <box size="0.059 0.041 0.029"/>
       </geometry>
       <material name="sensor_gray"/>
     </visual>
     <inertial>
-      <mass value="0.07"/>
-      <inertia ixx="0.0008" ixy="0" ixz="0" iyy="0.0008" iyz="0" izz="0.0008"/>
+      <mass value="0.058"/>
+      <inertia ixx="0.0006" ixy="0" ixz="0" iyy="0.0006" iyz="0" izz="0.0006"/>
     </inertial>
   </link>
@@ -205,10 +216,10 @@
   <gazebo reference="lidar_link">
     <sensor name="ydlidar_tg30" type="gpu_lidar">
-      <update_rate>5</update_rate>
+     <update_rate>2</update_rate>
       <topic>/scan</topic>
       <lidar>
         <scan>
           <horizontal>
-            <samples>720</samples>
+            <samples>360</samples>
             <resolution>1</resolution>
             <min_angle>-3.14159</min_angle>
@@ -226,13 +237,13 @@
     </sensor>
   </gazebo>
-  <gazebo reference="d435i_link">
-    <sensor name="d435i_depth" type="depth_camera">
-      <update_rate>10</update_rate>
-      <topic>/d435i/depth/image_raw</topic>
+  <gazebo reference="d435if_link">
+    <sensor name="d435if_depth" type="depth_camera">
+    <update_rate>2</update_rate>
+      <topic>/d435if/depth/image_raw</topic>
       <camera>
         <horizontal_fov>1.5184</horizontal_fov>
-        <image>
-          <width>640</width>
-          <height>480</height>
+       <image>
+      <width>320</width>
+      <height>240</height>
           <format>R8G8B8</format>
         </image>
@@ -248,11 +259,11 @@
   <gazebo reference="rpi_hq_camera_link">
     <sensor name="rpi_hq_camera" type="camera">
-      <update_rate>10</update_rate>
+      <update_rate>1</update_rate>
       <topic>/rpi_hq_camera/image_raw</topic>
       <camera>
         <horizontal_fov>0.6606</horizontal_fov>
         <image>
-          <width>640</width>
-          <height>480</height>
+          <width>320</width>
+  <height>240</height>
           <format>R8G8B8</format>
         </image>
@@ -266,24 +277,4 @@
     </sensor>
   </gazebo>
-  <gazebo reference="rear_camera_link">
-    <sensor name="rear_camera" type="camera">
-      <update_rate>5</update_rate>
-      <topic>/rear_camera/image_raw</topic>
-      <camera>
-        <horizontal_fov>1.5708</horizontal_fov>
-        <image>
-          <width>640</width>
-          <height>480</height>
-          <format>R8G8B8</format>
-        </image>
-        <clip>
-          <near>0.10</near>
-          <far>100.0</far>
-        </clip>
-      </camera>
-      <always_on>true</always_on>
-      <visualize>false</visualize>
-    </sensor>
-  </gazebo>
   <gazebo reference="wheel_fl">
     <mu1>1.0</mu1>

Commit message: Update sensor poses and finalize slalom notes

File: src/tulpar_description/urdf/robot.urdf.xacro (robot description, xacro)
@@ -84,5 +84,5 @@
     <parent link="base_link"/>
     <child link="lidar_link"/>
-    <origin xyz="0.30 0.0 0.40" rpy="0 0 0"/>
+    <origin xyz="0.58 -0.015 0.61" rpy="0 0 0"/>
   </joint>
   <link name="laser_frame"/>
@@ -108,5 +108,5 @@
     <parent link="base_link"/>
     <child link="d435if_link"/>
-    <origin xyz="0.62 0.0 0.20" rpy="0 0 0"/>
+    <origin xyz="0.58 0.0 0.53" rpy="0 0 0"/>
   </joint>
   <link name="d435if_color_frame"/>
@@ -158,5 +158,5 @@
     <parent link="base_link"/>
     <child link="rpi_hq_camera_link"/>
-    <origin xyz="0.58 0.0 0.28" rpy="0 0 0"/>
+    <origin xyz="0.58 -0.03 0.58" rpy="0 0 0"/>
   </joint>
   <link name="rpi_hq_camera_optical_frame"/>

Commit message: feat(urdf): mekanik olculerine gore parametreler guncellendi (65kg, r=0.20, sep=1.16)

File: src/tulpar_description/urdf/robot.urdf.xacro (robot description, xacro)
@@ -17,5 +17,5 @@
     <parent link="base_footprint"/>
     <child link="base_link"/>
-    <origin xyz="0 0 0.165" rpy="0 0 0"/>
+    <origin xyz="0 0 0.200" rpy="0 0 0"/>
   </joint>
   <link name="base_link">
@@ -30,11 +30,11 @@
       <origin xyz="0 0 0.1925" rpy="0 0 0"/>
       <geometry>
-        <box size="1.316 1.207 0.615"/>
+        <box size="1.150 1.207 0.615"/>
       </geometry>
     </collision>
     <inertial>
-      <mass value="60.0"/>
+      <mass value="65.0"/>
       <origin xyz="0 0 0" rpy="0 0 0"/>
-      <inertia ixx="8.520" ixy="0.0" ixz="0.0" iyy="22.140" iyz="0.0" izz="27.180"/>
+      <inertia ixx="9.94" ixy="0.0" ixz="0.0" iyy="9.21" iyz="0.0" izz="15.06"/>
     </inertial>
   </link>
@@ -49,10 +49,10 @@
       <collision>
         <geometry>
-          <cylinder radius="0.165" length="0.12"/>
+          <cylinder radius="0.20" length="0.12"/>
         </geometry>
       </collision>
       <inertial>
         <mass value="3.5"/>
-        <inertia ixx="0.024" ixy="0" ixz="0" iyy="0.024" iyz="0" izz="0.048"/>
+        <inertia ixx="0.039" ixy="0" ixz="0" iyy="0.039" iyz="0" izz="0.070"/>
       </inertial>
     </link>
@@ -65,8 +65,8 @@
     </joint>
   </xacro:macro>
-  <xacro:wheel name="wheel_fl" x="0.4" y="0.52"/>
-  <xacro:wheel name="wheel_rl" x="-0.4" y="0.52"/>
-  <xacro:wheel name="wheel_fr" x="0.4" y="-0.52"/>
-  <xacro:wheel name="wheel_rr" x="-0.4" y="-0.52"/>
+  <xacro:wheel name="wheel_fl" x="0.4" y="0.58"/>
+  <xacro:wheel name="wheel_rl" x="-0.4" y="0.58"/>
+  <xacro:wheel name="wheel_fr" x="0.4" y="-0.58"/>
+  <xacro:wheel name="wheel_rr" x="-0.4" y="-0.58"/>
   <link name="lidar_link">
     <visual>
@@ -201,6 +201,6 @@
       <right_joint>joint_wheel_fr</right_joint>
       <right_joint>joint_wheel_rr</right_joint>
-      <wheel_separation>1.04</wheel_separation>
-      <wheel_radius>0.165</wheel_radius>
+      <wheel_separation>1.16</wheel_separation>
+      <wheel_radius>0.20</wheel_radius>
       <max_linear_velocity>1.0</max_linear_velocity>
       <max_angular_velocity>3.0</max_angular_velocity>

Commit message: feat(mesh): govde tulpar_yeni.stl'e gecirildi, eski assembly mesh silindi (143MB)

File: src/tulpar_description/urdf/robot.urdf.xacro (robot description, xacro)
@@ -23,5 +23,5 @@
       <origin xyz="0.600 -0.300 0.110" rpy="0 0 1.5708"/>
       <geometry>
-        <mesh filename="package://tulpar_description/meshes/tulpar_ika_assembly.stl" scale="0.001 0.001 0.001"/>
+        <mesh filename="package://tulpar_description/meshes/tulpar_yeni.stl" scale="0.001 0.001 0.001"/>
       </geometry>
       <material name="aluminium"/>

Commit message: feat(mesh): govde mekanigin son tasarimina (tulpar_govde_final) gecirildi, origin ayarlandi

File: src/tulpar_description/urdf/robot.urdf.xacro (robot description, xacro)
@@ -21,7 +21,7 @@
   <link name="base_link">
     <visual>
-      <origin xyz="0.600 -0.300 0.110" rpy="0 0 1.5708"/>
-      <geometry>
-        <mesh filename="package://tulpar_description/meshes/tulpar_yeni.stl" scale="0.001 0.001 0.001"/>
+      <origin xyz="0.592 -0.225 0.110" rpy="0 0 1.5708"/>
+      <geometry>
+        <mesh filename="package://tulpar_description/meshes/tulpar_govde_final.stl" scale="0.001 0.001 0.001"/>
       </geometry>
       <material name="aluminium"/>
